Commit message: Explicit box inertia origin

File: xacro/box_inertia.xacro (robot description, xacro)
@@ -2,6 +2,7 @@
 <!-- SPDX-License-Identifier: Apache-2.0 -->
 <robot name="utils" xmlns:xacro="http://ros.org/wiki/xacro">
-    <xacro:macro name="box_inertia" params="len_x len_y len_z mass">
+    <xacro:macro name="box_inertia" params="len_x len_y len_z mass rpy xyz">
         <inertial>
+            <origin rpy="${rpy}" xyz="${xyz}" />
             <mass value="${mass}"/>
             <inertia

File: xacro/upkie.xacro (robot description, xacro)
@@ -73,5 +73,8 @@
         </collision>
         <!-- torso mass evaluated as net mass (5.4 [kg]) minus everything else -->
-        <xacro:box_inertia mass="1" len_x="0.125" len_y="0.17" len_z="0.25" />
+        <xacro:box_inertia
+            rpy="0 0 0" xyz="0 0 0"
+            mass="1"
+            len_x="0.125" len_y="0.17" len_z="0.25" />
     </link>
     <joint name="torso_fix" type="fixed">
@@ -94,5 +97,8 @@
         </collision>
         <!-- mass measurement was imprecise -->
-        <xacro:box_inertia mass="0.8" len_x="0.13" len_y="0.074" len_z="0.055" />
+        <xacro:box_inertia
+            rpy="0 0 0" xyz="0 0 0"
+            mass="0.8"
+            len_x="0.13" len_y="0.074" len_z="0.055" />
     </link>
     <joint name="battery_fix" type="fixed">
