Commit message: Avoid inline comments to ease conversion checks

File: xacro/upkie.xacro (robot description, xacro)
@@ -36,6 +36,8 @@
     </material>
     <link name="base">
-        <inertial>  <!-- virtual -->
-            <mass value="0.001" />  <!-- not zero, see [1] -->
+        <!-- virtual link -->
+        <inertial>
+            <!-- mass should not be zero [1] -->
+            <mass value="0.001" />
             <origin rpy="0 0 0" xyz="0 0 0" />
             <inertia ixx="0" ixy="0" ixz="0" iyy="0" iyz="0" izz="0" />
@@ -44,6 +46,8 @@
     <!-- IMU -->
     <link name="imu">
-        <inertial>  <!-- virtual -->
-            <mass value="0.001" />  <!-- not zero, see [1] -->
+        <!-- virtual link -->
+        <inertial>
+            <!-- mass should not be zero [1] -->
+            <mass value="0.001" />
             <origin rpy="0 0 0" xyz="0 0 0" />
             <inertia ixx="0" ixy="0" ixz="0" iyy="0" iyz="0" izz="0" />
@@ -69,5 +73,6 @@
         </collision>
         <inertial>
-            <mass value="1.0" />  <!-- measured net mass (5.4 [kg]) minus everything else -->
+            <!-- torso mass evaluated as net mass (5.4 [kg]) minus everything else -->
+            <mass value="1.0" />
             <!-- ./box_inertia.py 1.0 0.125 0.17 0.25 -->
             <inertia ixx="0.007616666666666667" ixy="0" ixz="0" iyx="0" iyy="0.006510416666666666" iyz="0" izx="0" izy="0" izz="0.0037104166666666674" />
@@ -119,5 +124,6 @@
         <inertial>
             <origin rpy="0 0 0" xyz="0 0 0.01" />
-            <mass value="0.0525" />  <!-- measured -->
+            <!-- mass measured on a real robot -->
+            <mass value="0.0525" />
             <!-- ./box_inertia.py 0.0525 0.120 0.07 0.04 -->
             <inertia ixx="2.84375e-05" ixy="0" ixz="0" iyx="0" iyy="7e-05" iyz="0" izx="0" izy="0" izz="8.44375e-05" />
@@ -198,5 +204,6 @@
         <inertial>
             <origin rpy="0 1.5707963267948966 0" xyz="0 0 0.025" />
-            <mass value="0.05267" />  <!-- measured, with screws -->
+            <!-- mass measured with screws -->
+            <mass value="0.05267" />
             <!-- ./cylinder_inertia.py 0.05267 0.025 0.09 -->
             <inertia ixx="4.37819375e-05" ixy="0" ixz="0" iyx="0" iyy="4.37819375e-05" iyz="0" izx="0" izy="0" izz="1.6459375e-05" />
@@ -223,5 +230,6 @@
         </collision>
         <inertial>
-            <mass value="0.056" />  <!-- measured, average over four sticks -->
+            <!-- mass measured on average over four wooden sticks -->
+            <mass value="0.056" />
             <!-- ./cylinder_inertia.py 0.056 0.012 0.026 -->
             <inertia ixx="5.170666666666667e-06" ixy="0" ixz="0" iyx="0" iyy="5.170666666666667e-06" iyz="0" izx="0" izy="0" izz="4.0320000000000005e-06" />
@@ -326,5 +334,6 @@
         <inertial>
             <origin rpy="0 1.5707963267948966 0" xyz="0 0 0.025" />
-            <mass value="0.05267" />  <!-- measured, with screws -->
+            <!-- mass measured with screws -->
+            <mass value="0.05267" />
             <!-- ./cylinder_inertia.py 0.05267 0.025 0.09 -->
             <inertia ixx="4.37819375e-05" ixy="0" ixz="0" iyx="0" iyy="4.37819375e-05" iyz="0" izx="0" izy="0" izz="1.6459375e-05" />
@@ -351,5 +360,6 @@
         </collision>
         <inertial>
-            <mass value="0.056" />  <!-- measured, average over four sticks -->
+            <!-- mass measured on average over four wooden sticks -->
+            <mass value="0.056" />
             <!-- ./cylinder_inertia.py 0.056 0.012 0.026 -->
             <inertia ixx="5.170666666666667e-06" ixy="0" ixz="0" iyx="0" iyy="5.170666666666667e-06" iyz="0" izx="0" izy="0" izz="4.0320000000000005e-06" />
@@ -377,5 +387,6 @@
         <inertial>
             <origin rpy="0 0 0" xyz="0 0.002 0.0275" />
-            <mass value="0.07863" />  <!-- measured, with screws -->
+            <!-- mass measured with screws -->
+            <mass value="0.07863" />
             <!-- ./box_inertia.py 0.07863 0.092 0.068 0.056 -->
             <inertia ixx="5.084740000000001e-05" ixy="0" ixz="0" iyx="0" iyy="7.6009e-05" iyz="0" izx="0" izy="0" izz="8.575912e-05" />
@@ -425,5 +436,6 @@
         <inertial>
             <origin rpy="0 0 0" xyz="0 0 0.01" />
-            <mass value="0.1721" />  <!-- measured 242.1 [g], minus 20 [g] for the plate, minus 50 [g] for the rotor -->
+            <!-- mass measured was 242.1 [g], minus 20 [g] for the plate, minus 50 [g] for the rotor -->
+            <mass value="0.1721" />
             <!-- ./cylinder_inertia.py 0.1721 0.03 0.018 -->
             <inertia ixx="4.3369200000000005e-05" ixy="0" ixz="0" iyx="0" iyy="4.3369200000000005e-05" iyz="0" izx="0" izy="0" izz="7.7445e-05" />
@@ -436,6 +448,8 @@
     </joint>
     <link name="left_anchor">
-        <inertial>  <!-- virtual -->
-            <mass value="0.001" />  <!-- not zero, see [1] -->
+        <!-- virtual link -->
+        <inertial>
+            <!-- mass should not be zero [1] -->
+            <mass value="0.001" />
             <origin rpy="0 0 0" xyz="0 0 0" />
             <inertia ixx="0" ixy="0" ixz="0" iyy="0" iyz="0" izz="0" />
@@ -490,5 +504,6 @@
         <inertial>
             <origin rpy="0 0 0" xyz="0 0 0.0125" />
-            <mass value="0.0454" />  <!-- measured, with hub adapter -->
+            <!-- mass measured with hub adapter -->
+            <mass value="0.0454" />
             <!-- ./cylinder_inertia.py 0.0454 0.039 0.025 -->
             <inertia ixx="1.9627933333333332e-05" ixy="0" ixz="0" iyx="0" iyy="1.9627933333333332e-05" iyz="0" izx="0" izy="0" izz="3.45267e-05" />
@@ -513,5 +528,6 @@
         </collision>
         <inertial>
-            <mass value="0.08715" />  <!-- measured -->
+            <!-- mass measured on a real robot -->
+            <mass value="0.08715" />
             <!-- ./cylinder_inertia.py 0.08715 0.05 0.04 -->
             <inertia ixx="6.608875000000002e-05" ixy="0" ixz="0" iyx="0" iyy="6.608875000000002e-05" iyz="0" izx="0" izy="0" izz="0.00010893750000000003" />
@@ -530,6 +546,8 @@
     </joint>
     <link name="left_contact">
-        <inertial>  <!-- virtual -->
-            <mass value="0.001" />  <!-- not zero, see [1] -->
+        <!-- virtual link -->
+        <inertial>
+            <!-- mass should not be zero [1] -->
+            <mass value="0.001" />
             <origin rpy="0 0 0" xyz="0 0 0" />
             <inertia ixx="0" ixy="0" ixz="0" iyy="0" iyz="0" izz="0" />
@@ -544,6 +562,8 @@
     </joint>
     <link name="left_wheel_center">
-        <inertial>  <!-- virtual -->
-            <mass value="0.001" />  <!-- not zero, see [1] -->
+        <!-- virtual link -->
+        <inertial>
+            <!-- mass should not be zero [1] -->
+            <mass value="0.001" />
             <origin rpy="0 0 0" xyz="0 0 0" />
             <inertia ixx="0" ixy="0" ixz="0" iyy="0" iyz="0" izz="0" />
@@ -624,5 +644,6 @@
         <inertial>
             <origin rpy="0 1.5707963267948966 0" xyz="0 0 0.025" />
-            <mass value="0.05267" />  <!-- measured, with screws -->
+            <!-- mass measured with screws -->
+            <mass value="0.05267" />
             <!-- ./cylinder_inertia.py 0.05267 0.025 0.09 -->
             <inertia ixx="4.37819375e-05" ixy="0" ixz="0" iyx="0" iyy="4.37819375e-05" iyz="0" izx="0" izy="0" izz="1.6459375e-05" />
@@ -649,5 +670,6 @@
         </collision>
         <inertial>
-            <mass value="0.056" />  <!-- measured, average over four sticks -->
+            <!-- mass measured on average over four wooden sticks -->
+            <mass value="0.056" />
             <!-- ./cylinder_inertia.py 0.056 0.012 0.026 -->
             <inertia ixx="5.170666666666667e-06" ixy="0" ixz="0" iyx="0" iyy="5.170666666666667e-06" iyz="0" izx="0" izy="0" izz="4.0320000000000005e-06" />
@@ -752,5 +774,6 @@
         <inertial>
             <origin rpy="0 1.5707963267948966 0" xyz="0 0 0.025" />
-            <mass value="0.05267" />  <!-- measured, with screws -->
+            <!-- mass measured with screws -->
+            <mass value="0.05267" />
             <!-- ./cylinder_inertia.py 0.05267 0.025 0.09 -->
             <inertia ixx="4.37819375e-05" ixy="0" ixz="0" iyx="0" iyy="4.37819375e-05" iyz="0" izx="0" izy="0" izz="1.6459375e-05" />
@@ -777,5 +800,6 @@
         </collision>
         <inertial>
-            <mass value="0.056" />  <!-- measured, average over four sticks -->
+            <!-- mass measured on average over four wooden sticks -->
+            <mass value="0.056" />
             <!-- ./cylinder_inertia.py 0.056 0.012 0.026 -->
             <inertia ixx="5.170666666666667e-06" ixy="0" ixz="0" iyx="0" iyy="5.170666666666667e-06" iyz="0" izx="0" izy="0" izz="4.0320000000000005e-06" />
@@ -803,5 +827,6 @@
         <inertial>
             <origin rpy="0 0 0" xyz="0 0.002 0.0275" />
-            <mass value="0.07863" />  <!-- measured, with screws -->
+            <!-- mass measured with screws -->
+            <mass value="0.07863" />
             <!-- ./box_inertia.py 0.07863 0.092 0.068 0.056 -->
             <inertia ixx="5.084740000000001e-05" ixy="0" ixz="0" iyx="0" iyy="7.6009e-05" iyz="0" izx="0" izy="0" izz="8.575912e-05" />
@@ -851,5 +876,6 @@
         <inertial>
             <origin rpy="0 0 0" xyz="0 0 0.01" />
-            <mass value="0.1721" />  <!-- measured 242.1 [g], minus 20 [g] for the plate, minus 50 [g] for the rotor -->
+            <!-- mass measured was 242.1 [g], minus 20 [g] for the plate, minus 50 [g] for the rotor -->
+            <mass value="0.1721" />
             <!-- ./cylinder_inertia.py 0.1721 0.03 0.018 -->
             <inertia ixx="4.3369200000000005e-05" ixy="0" ixz="0" iyx="0" iyy="4.3369200000000005e-05" iyz="0" izx="0" izy="0" izz="7.7445e-05" />
@@ -862,6 +888,8 @@
     </joint>
     <link name="right_anchor">
-        <inertial>  <!-- virtual -->
-            <mass value="0.001" />  <!-- not zero, see [1] -->
+        <!-- virtual link -->
+        <inertial>
+            <!-- mass should not be zero [1] -->
+            <mass value="0.001" />
             <origin rpy="0 0 0" xyz="0 0 0" />
             <inertia ixx="0" ixy="0" ixz="0" iyy="0" iyz="0" izz="0" />
@@ -916,5 +944,6 @@
         <inertial>
             <origin rpy="0 0 0" xyz="0 0 0.0125" />
-            <mass value="0.0454" />  <!-- measured, with hub adapter -->
+            <!-- mass measured with hub adapter -->
+            <mass value="0.0454" />
             <!-- ./cylinder_inertia.py 0.0454 0.039 0.025 -->
             <inertia ixx="1.9627933333333332e-05" ixy="0" ixz="0" iyx="0" iyy="1.9627933333333332e-05" iyz="0" izx="0" izy="0" izz="3.45267e-05" />
@@ -939,5 +968,6 @@
         </collision>
         <inertial>
-            <mass value="0.08715" />  <!-- measured -->
+            <!-- mass measured on a real tire -->
+            <mass value="0.08715" />
             <!-- ./cylinder_inertia.py 0.08715 0.05 0.04 -->
             <inertia ixx="6.608875000000002e-05" ixy="0" ixz="0" iyx="0" iyy="6.608875000000002e-05" iyz="0" izx="0" izy="0" izz="0.00010893750000000003" />
@@ -956,6 +986,8 @@
     </joint>
     <link name="right_contact">
-        <inertial>  <!-- virtual -->
-            <mass value="0.001" />  <!-- not zero, see [1] -->
+        <!-- virtual link -->
+        <inertial>
+            <!-- mass should not be zero [1] -->
+            <mass value="0.001" />
             <origin rpy="0 0 0" xyz="0 0 0" />
             <inertia ixx="0" ixy="0" ixz="0" iyy="0" iyz="0" izz="0" />
@@ -970,6 +1002,8 @@
     </joint>
     <link name="right_wheel_center">
-        <inertial>  <!-- virtual -->
-            <mass value="0.001" />  <!-- not zero, see [1] -->
+        <!-- virtual link -->
+        <inertial>
+            <!-- mass should not be zero [1] -->
+            <mass value="0.001" />
             <origin rpy="0 0 0" xyz="0 0 0" />
             <inertia ixx="0" ixy="0" ixz="0" iyy="0" iyz="0" izz="0" />

Commit message: Swap cylinder radius and length attributes

File: xacro/upkie.xacro (robot description, xacro)
@@ -147,5 +147,5 @@
             <origin rpy="0 0 0" xyz="0 0 0.015" />
             <geometry>
-                <cylinder radius="0.05" length="0.03" />
+                <cylinder length="0.03" radius="0.05" />
             </geometry>
         </collision>
@@ -172,5 +172,5 @@
             <origin rpy="0 0 0" xyz="0 0 -0.0025" />
             <geometry>
-                <cylinder radius="0.023" length="0.005" />
+                <cylinder length="0.005" radius="0.023" />
             </geometry>
         </collision>
@@ -199,5 +199,5 @@
             <origin rpy="0 1.5707963267948966 0" xyz="0 0 0.025" />
             <geometry>
-                <cylinder radius="0.025" length="0.09" />
+                <cylinder length="0.09" radius="0.025" />
             </geometry>
         </collision>
@@ -225,5 +225,5 @@
         <collision>
             <geometry>
-                <cylinder radius="0.012" length="0.26" />
+                <cylinder length="0.26" radius="0.012" />
             </geometry>
             <material name="light_wood" />
@@ -257,5 +257,5 @@
             <origin rpy="0 1.5707963267948966 0" xyz="0.03 0 0" />
             <geometry>
-                <cylinder radius="0.05" length="0.06" />
+                <cylinder length="0.06" radius="0.05" />
             </geometry>
         </collision>
@@ -277,5 +277,5 @@
             <origin rpy="0 0 0" xyz="0 0 0.015" />
             <geometry>
-                <cylinder radius="0.05" length="0.03" />
+                <cylinder length="0.03" radius="0.05" />
             </geometry>
         </collision>
@@ -309,5 +309,5 @@
             <origin rpy="0 0 0" xyz="0 0 -0.0025" />
             <geometry>
-                <cylinder radius="0.023" length="0.005" />
+                <cylinder length="0.005" radius="0.023" />
             </geometry>
         </collision>
@@ -329,5 +329,5 @@
             <origin rpy="0 1.5707963267948966 0" xyz="0 0 0.025" />
             <geometry>
-                <cylinder radius="0.025" length="0.09" />
+                <cylinder length="0.09" radius="0.025" />
             </geometry>
         </collision>
@@ -355,5 +355,5 @@
         <collision>
             <geometry>
-                <cylinder radius="0.012" length="0.26" />
+                <cylinder length="0.26" radius="0.012" />
             </geometry>
             <material name="light_wood" />
@@ -431,5 +431,5 @@
             <origin rpy="0 0 0" xyz="0 0 0.01" />
             <geometry>
-                <cylinder radius="0.03" length="0.018" />
+                <cylinder length="0.018" radius="0.03" />
             </geometry>
         </collision>
@@ -471,5 +471,5 @@
             <origin rpy="0 0 0" xyz="0 0 0.015" />
             <geometry>
-                <cylinder radius="0.034" length="0.016" />
+                <cylinder length="0.016" radius="0.034" />
             </geometry>
         </collision>
@@ -499,5 +499,5 @@
             <origin rpy="0 0 0" xyz="0 0 0.0125" />
             <geometry>
-                <cylinder radius="0.039" length="0.025" />
+                <cylinder length="0.025" radius="0.039" />
             </geometry>
         </collision>
@@ -524,5 +524,5 @@
         <collision>
             <geometry>
-                <cylinder radius="0.05" length="0.04" />
+                <cylinder length="0.04" radius="0.05" />
             </geometry>
         </collision>
@@ -587,5 +587,5 @@
             <origin rpy="0 0 0" xyz="0 0 0.015" />
             <geometry>
-                <cylinder radius="0.05" length="0.03" />
+                <cylinder length="0.03" radius="0.05" />
             </geometry>
         </collision>
@@ -612,5 +612,5 @@
             <origin rpy="0 0 0" xyz="0 0 -0.0025" />
             <geometry>
-                <cylinder radius="0.023" length="0.005" />
+                <cylinder length="0.005" radius="0.023" />
             </geometry>
         </collision>
@@ -639,5 +639,5 @@
             <origin rpy="0 1.5707963267948966 0" xyz="0 0 0.025" />
             <geometry>
-                <cylinder radius="0.025" length="0.09" />
+                <cylinder length="0.09" radius="0.025" />
             </geometry>
         </collision>
@@ -665,5 +665,5 @@
         <collision>
             <geometry>
-                <cylinder radius="0.012" length="0.26" />
+                <cylinder length="0.26" radius="0.012" />
             </geometry>
             <material name="light_wood" />
@@ -697,5 +697,5 @@
             <origin rpy="0 1.5707963267948966 0" xyz="0.03 0 0" />
             <geometry>
-                <cylinder radius="0.05" length="0.06" />
+                <cylinder length="0.06" radius="0.05" />
             </geometry>
         </collision>
@@ -717,5 +717,5 @@
             <origin rpy="0 0 0" xyz="0 0 0.015" />
             <geometry>
-                <cylinder radius="0.05" length="0.03" />
+                <cylinder length="0.03" radius="0.05" />
             </geometry>
         </collision>
@@ -749,5 +749,5 @@
             <origin rpy="0 0 0" xyz="0 0 -0.0025" />
             <geometry>
-                <cylinder radius="0.023" length="0.005" />
+                <cylinder length="0.005" radius="0.023" />
             </geometry>
         </collision>
@@ -769,5 +769,5 @@
             <origin rpy="0 1.5707963267948966 0" xyz="0 0 0.025" />
             <geometry>
-                <cylinder radius="0.025" length="0.09" />
+                <cylinder length="0.09" radius="0.025" />
             </geometry>
         </collision>
@@ -795,5 +795,5 @@
         <collision>
             <geometry>
-                <cylinder radius="0.012" length="0.26" />
+                <cylinder length="0.26" radius="0.012" />
             </geometry>
             <material name="light_wood" />
@@ -871,5 +871,5 @@
             <origin rpy="0 0 0" xyz="0 0 0.01" />
             <geometry>
-                <cylinder radius="0.03" length="0.018" />
+                <cylinder length="0.018" radius="0.03" />
             </geometry>
         </collision>
@@ -911,5 +911,5 @@
             <origin rpy="0 0 0" xyz="0 0 0.015" />
             <geometry>
-                <cylinder radius="0.034" length="0.016" />
+                <cylinder length="0.016" radius="0.034" />
             </geometry>
         </collision>
@@ -939,5 +939,5 @@
             <origin rpy="0 0 0" xyz="0 0 0.0125" />
             <geometry>
-                <cylinder radius="0.039" length="0.025" />
+                <cylinder length="0.025" radius="0.039" />
             </geometry>
         </collision>
@@ -964,5 +964,5 @@
         <collision>
             <geometry>
-                <cylinder radius="0.05" length="0.04" />
+                <cylinder length="0.04" radius="0.05" />
             </geometry>
         </collision>
