Commit message: No inline comment, continued

File: xacro/upkie.xacro (robot description, xacro)
@@ -55,5 +55,6 @@
     </link>
     <joint name="imu_fix" type="fixed">
-        <origin rpy="3.141592653589793 0 3.141592653589793" xyz="0 0 0" />  <!-- no translation -->
+        <!-- not that the origin frame is not translated -->
+        <origin rpy="3.141592653589793 0 3.141592653589793" xyz="0 0 0" />
         <parent link="base" />
         <child link="imu" />
@@ -98,5 +99,6 @@
         </collision>
         <inertial>
-            <mass value="0.800" />  <!-- imprecise measurement -->
+            <!-- mass measurement was imprecise -->
+            <mass value="0.8" />
             <!-- ./box_inertia.py 0.800 0.13 0.074 0.055 -->
             <inertia ixx="0.0005667333333333332" ixy="0" ixz="0" iyx="0" iyy="0.0013283333333333335" iyz="0" izx="0" izy="0" izz="0.0014917333333333332" />
@@ -152,5 +154,6 @@
         <inertial>
             <origin rpy="0 0 0" xyz="0 0 0.015" />
-            <mass value="0.47" />  <!-- guessed from spec -->
+            <!-- mass guessed from spec -->
+            <mass value="0.47" />
             <!-- ./cylinder_inertia.py 0.470 0.05 0.03 -->
             <inertia ixx="0.000329" ixy="0" ixz="0" iyx="0" iyy="0.000329" iyz="0" izx="0" izy="0" izz="0.0005875" />
@@ -177,5 +180,6 @@
         <inertial>
             <origin rpy="0 0 0" xyz="0 0 -0.0025" />
-            <mass value="0.015" />  <!-- guessed from spec -->
+            <!-- mass guessed from spec -->
+            <mass value="0.015" />
             <!-- ./cylinder_inertia.py 0.015 0.023 0.005 -->
             <inertia ixx="2.0149999999999998e-06" ixy="0" ixz="0" iyx="0" iyy="2.0149999999999998e-06" iyz="0" izx="0" izy="0" izz="3.9675e-06" />
@@ -186,5 +190,6 @@
         <child link="left_hip_qdd100_rotor" />
         <origin rpy="0 0 0" xyz="0 0 0.0292" />
-        <axis xyz="0 0 -1" />  <!-- search "moteus-direction-configuration" -->
+        <!-- negative z-axis: search "moteus-direction-configuration" -->
+        <axis xyz="0 0 -1" />
         <limit lower="-1.26" upper="1.26" velocity="28.8" effort="16.0" />
     </joint>
@@ -262,5 +267,6 @@
         <inertial>
             <origin rpy="0 1.5707963267948966 0" xyz="0.03 0 0" />
-            <mass value="0.09874" />  <!-- Used Filament estimate from Prusa Slicer -->
+            <!-- mass based on filament estimate from Prusa Slicer -->
+            <mass value="0.09874" />
             <!-- ./cylinder_inertia.py 0.09874 0.05 0.06 -->
             <inertia ixx="9.133450000000001e-05" ixy="0" ixz="0" iyx="0" iyy="9.133450000000001e-05" iyz="0" izx="0" izy="0" izz="0.000123425" />
@@ -282,5 +288,6 @@
         <inertial>
             <origin rpy="0 0 0" xyz="0 0 0.015" />
-            <mass value="0.47" />  <!-- guessed from spec -->
+            <!-- mass guessed from spec -->
+            <mass value="0.47" />
             <!-- ./cylinder_inertia.py 0.470 0.05 0.03 -->
             <inertia ixx="0.000329" ixy="0" ixz="0" iyx="0" iyy="0.000329" iyz="0" izx="0" izy="0" izz="0.0005875" />
@@ -296,5 +303,6 @@
         <child link="left_knee_qdd100_rotor" />
         <origin rpy="0 0 0" xyz="0 0 0.0292" />
-        <axis xyz="0 0 -1" />  <!-- search "moteus-direction-configuration" -->
+        <!-- negative z-axis: search "moteus-direction-configuration" -->
+        <axis xyz="0 0 -1" />
         <limit lower="-2.51" upper="2.51" velocity="28.8" effort="16.0" />
     </joint>
@@ -314,5 +322,6 @@
         <inertial>
             <origin rpy="0 0 0" xyz="0 0 -0.0025" />
-            <mass value="0.015" />  <!-- guessed from spec -->
+            <!-- mass guessed from spec -->
+            <mass value="0.015" />
             <!-- ./cylinder_inertia.py 0.015 0.023 0.005 -->
             <inertia ixx="2.0149999999999998e-06" ixy="0" ixz="0" iyx="0" iyy="2.0149999999999998e-06" iyz="0" izx="0" izy="0" izz="3.9675e-06" />
@@ -411,5 +420,6 @@
         </collision>
         <inertial>
-            <mass value="0.02" />  <!-- pure guess (^_^") -->
+            <!-- mass is a pure guess (^_^") -->
+            <mass value="0.02" />
             <!-- ./box_inertia.py 0.02 0.09 0.046 0.004 -->
             <inertia ixx="3.5533333333333333e-06" ixy="0" ixz="0" iyx="0" iyy="1.3526666666666667e-05" iyz="0" izx="0" izy="0" izz="1.7026666666666667e-05" />
@@ -476,5 +486,6 @@
         <inertial>
             <origin rpy="0 0 0" xyz="0 0 0.015" />
-            <mass value="0.05" />  <!-- guess at 50 [g] for the rotor -->
+            <!-- mass is a pure guess -->
+            <mass value="0.05" />
             <!-- ./cylinder_inertia.py 0.05 0.034 0.016 -->
             <inertia ixx="1.551666666666667e-05" ixy="0" ixz="0" iyx="0" iyy="1.551666666666667e-05" iyz="0" izx="0" izy="0" izz="2.8900000000000005e-05" />
@@ -485,5 +496,6 @@
         <child link="left_ankle_mj5208_rotor" />
         <origin rpy="0 0 0" xyz="0 0 0" />
-        <axis xyz="0 0 -1" />  <!-- search "moteus-direction-configuration" -->
+        <!-- negative z-axis: search "moteus-direction-configuration" -->
+        <axis xyz="0 0 -1" />
         <limit velocity="111.0" effort="1.7" />
     </joint>
@@ -592,5 +604,6 @@
         <inertial>
             <origin rpy="0 0 0" xyz="0 0 0.015" />
-            <mass value="0.47" />  <!-- guessed from spec -->
+            <!-- mass guessed from spec -->
+            <mass value="0.47" />
             <!-- ./cylinder_inertia.py 0.470 0.05 0.03 -->
             <inertia ixx="0.000329" ixy="0" ixz="0" iyx="0" iyy="0.000329" iyz="0" izx="0" izy="0" izz="0.0005875" />
@@ -617,5 +630,6 @@
         <inertial>
             <origin rpy="0 0 0" xyz="0 0 -0.0025" />
-            <mass value="0.015" />  <!-- guessed from spec -->
+            <!-- mass guessed from spec -->
+            <mass value="0.015" />
             <!-- ./cylinder_inertia.py 0.015 0.023 0.005 -->
             <inertia ixx="2.0149999999999998e-06" ixy="0" ixz="0" iyx="0" iyy="2.0149999999999998e-06" iyz="0" izx="0" izy="0" izz="3.9675e-06" />
@@ -626,5 +640,6 @@
         <child link="right_hip_qdd100_rotor" />
         <origin rpy="0 0 0" xyz="0 0 0.0292" />
-        <axis xyz="0 0 -1" />  <!-- search "moteus-direction-configuration" -->
+        <!-- negative z-axis: search "moteus-direction-configuration" -->
+        <axis xyz="0 0 -1" />
         <limit lower="-1.26" upper="1.26" velocity="28.8" effort="16.0" />
     </joint>
@@ -702,5 +717,6 @@
         <inertial>
             <origin rpy="0 1.5707963267948966 0" xyz="0.03 0 0" />
-            <mass value="0.09874" />  <!-- Used Filament estimate from Prusa Slicer -->
+            <!-- mass based on filament estimate from Prusa Slicer -->
+            <mass value="0.09874" />
             <!-- ./cylinder_inertia.py 0.09874 0.05 0.06 -->
             <inertia ixx="9.133450000000001e-05" ixy="0" ixz="0" iyx="0" iyy="9.133450000000001e-05" iyz="0" izx="0" izy="0" izz="0.000123425" />
@@ -722,5 +738,6 @@
         <inertial>
             <origin rpy="0 0 0" xyz="0 0 0.015" />
-            <mass value="0.47" />  <!-- guessed from spec -->
+            <!-- mass guessed from spec -->
+            <mass value="0.47" />
             <!-- ./cylinder_inertia.py 0.470 0.05 0.03 -->
             <inertia ixx="0.000329" ixy="0" ixz="0" iyx="0" iyy="0.000329" iyz="0" izx="0" izy="0" izz="0.0005875" />
@@ -736,5 +753,6 @@
         <child link="right_knee_qdd100_rotor" />
         <origin rpy="0 0 0" xyz="0 0 0.0292" />
-        <axis xyz="0 0 -1" />  <!-- search "moteus-direction-configuration" -->
+        <!-- negative z-axis: search "moteus-direction-configuration" -->
+        <axis xyz="0 0 -1" />
         <limit lower="-2.51" upper="2.51" velocity="28.8" effort="16.0" />
     </joint>
@@ -754,5 +772,6 @@
         <inertial>
             <origin rpy="0 0 0" xyz="0 0 -0.0025" />
-            <mass value="0.015" />  <!-- guessed from spec -->
+            <!-- mass guessed from spec -->
+            <mass value="0.015" />
             <!-- ./cylinder_inertia.py 0.015 0.023 0.005 -->
             <inertia ixx="2.0149999999999998e-06" ixy="0" ixz="0" iyx="0" iyy="2.0149999999999998e-06" iyz="0" izx="0" izy="0" izz="3.9675e-06" />
@@ -851,5 +870,6 @@
         </collision>
         <inertial>
-            <mass value="0.02" />  <!-- pure guess (^_^") -->
+            <!-- mass is a pure guess (^_^") -->
+            <mass value="0.02" />
             <!-- ./box_inertia.py 0.02 0.09 0.046 0.004 -->
             <inertia ixx="3.5533333333333333e-06" ixy="0" ixz="0" iyx="0" iyy="1.3526666666666667e-05" iyz="0" izx="0" izy="0" izz="1.7026666666666667e-05" />
@@ -916,5 +936,6 @@
         <inertial>
             <origin rpy="0 0 0" xyz="0 0 0.015" />
-            <mass value="0.05" />  <!-- guess at 50 [g] for the rotor -->
+            <!-- mass is a pure guess -->
+            <mass value="0.05" />
             <!-- ./cylinder_inertia.py 0.05 0.034 0.016 -->
             <inertia ixx="1.551666666666667e-05" ixy="0" ixz="0" iyx="0" iyy="1.551666666666667e-05" iyz="0" izx="0" izy="0" izz="2.8900000000000005e-05" />
@@ -925,5 +946,6 @@
         <child link="right_ankle_mj5208_rotor" />
         <origin rpy="0 0 0" xyz="0 0 0" />
-        <axis xyz="0 0 -1" />  <!-- search "moteus-direction-configuration" -->
+        <!-- negative z-axis: search "moteus-direction-configuration" -->
+        <axis xyz="0 0 -1" />
         <limit velocity="111.0" effort="1.7" />
     </joint>

Commit message: Sort limit attributes alphabetically

File: xacro/upkie.xacro (robot description, xacro)
@@ -3,8 +3,6 @@
 <!-- Copyright 2022 Stéphane Caron -->
 <!-- Copyright 2023 Inria -->
-<!--
-Conventions in this file are detailed in:
-https://github.com/upkie/upkie_description/wiki/Model-conventions
--->
+<!-- This file was generated from upkie.xacro -->
+<!-- Conventions in this file are detailed in: https://github.com/upkie/upkie_description/wiki/ -->
 <robot name="upkie">
     <material name="black">
@@ -192,5 +190,5 @@
         <!-- negative z-axis: search "moteus-direction-configuration" -->
         <axis xyz="0 0 -1" />
-        <limit lower="-1.26" upper="1.26" velocity="28.8" effort="16.0" />
+        <limit effort="16.0" lower="-1.26" upper="1.26" velocity="28.8" />
     </joint>
     <link name="left_hip_horn">
@@ -305,5 +303,5 @@
         <!-- negative z-axis: search "moteus-direction-configuration" -->
         <axis xyz="0 0 -1" />
-        <limit lower="-2.51" upper="2.51" velocity="28.8" effort="16.0" />
+        <limit effort="16.0" lower="-2.51" upper="2.51" velocity="28.8" />
     </joint>
     <link name="left_knee_qdd100_rotor">
@@ -498,5 +496,5 @@
         <!-- negative z-axis: search "moteus-direction-configuration" -->
         <axis xyz="0 0 -1" />
-        <limit velocity="111.0" effort="1.7" />
+        <limit effort="1.7" velocity="111.0" />
     </joint>
     <!-- Left wheel -->
@@ -642,5 +640,5 @@
         <!-- negative z-axis: search "moteus-direction-configuration" -->
         <axis xyz="0 0 -1" />
-        <limit lower="-1.26" upper="1.26" velocity="28.8" effort="16.0" />
+        <limit effort="16.0" lower="-1.26" upper="1.26" velocity="28.8" />
     </joint>
     <link name="right_hip_horn">
@@ -755,5 +753,5 @@
         <!-- negative z-axis: search "moteus-direction-configuration" -->
         <axis xyz="0 0 -1" />
-        <limit lower="-2.51" upper="2.51" velocity="28.8" effort="16.0" />
+        <limit effort="16.0" lower="-2.51" upper="2.51" velocity="28.8" />
     </joint>
     <link name="right_knee_qdd100_rotor">
@@ -948,5 +946,5 @@
         <!-- negative z-axis: search "moteus-direction-configuration" -->
         <axis xyz="0 0 -1" />
-        <limit velocity="111.0" effort="1.7" />
+        <limit effort="1.7" velocity="111.0" />
     </joint>
     <!-- Right wheel -->
@@ -1037,4 +1035,5 @@
         <origin rpy="1.5707963267948966 3.141592653589793 0" xyz="0 0 0" />
     </joint>
+</robot>
 <!--
 Footnotes:
@@ -1044,3 +1043,2 @@
 significant difference.
 -->
-</robot>
