Commit message: Move comments outside of inertial tags

File: xacro/upkie.xacro (robot description, xacro)
@@ -93,6 +93,6 @@
             </geometry>
         </collision>
-        <inertial>
-            <!-- mass measurement was imprecise -->
+        <!-- mass measurement was imprecise -->
+        <inertial>
             <mass value="0.8" />
             <!-- ./box_inertia.py 0.800 0.13 0.074 0.055 -->
@@ -119,7 +119,7 @@
             </geometry>
         </collision>
+        <!-- mass measured on a real robot -->
         <inertial>
             <origin rpy="0 0 0" xyz="0 0 0.01" />
-            <!-- mass measured on a real robot -->
             <mass value="0.0525" />
             <!-- ./box_inertia.py 0.0525 0.120 0.07 0.04 -->
@@ -147,7 +147,7 @@
             </geometry>
         </collision>
-        <inertial>
-            <origin rpy="0 0 0" xyz="0 0 0.015" />
-            <!-- mass guessed from spec -->
+        <!-- mass guessed from spec -->
+        <inertial>
+            <origin rpy="0 0 0" xyz="0 0 0.015" />
             <mass value="0.47" />
             <!-- ./cylinder_inertia.py 0.470 0.05 0.03 -->
@@ -173,7 +173,7 @@
             </geometry>
         </collision>
+        <!-- mass guessed from spec -->
         <inertial>
             <origin rpy="0 0 0" xyz="0 0 -0.0025" />
-            <!-- mass guessed from spec -->
             <mass value="0.015" />
             <!-- ./cylinder_inertia.py 0.015 0.023 0.005 -->
@@ -202,7 +202,7 @@
             </geometry>
         </collision>
+        <!-- mass measured with screws -->
         <inertial>
             <origin rpy="0 1.5707963267948966 0" xyz="0 0 0.025" />
-            <!-- mass measured with screws -->
             <mass value="0.05267" />
             <!-- ./cylinder_inertia.py 0.05267 0.025 0.09 -->
@@ -229,6 +229,6 @@
             <material name="light_wood" />
         </collision>
-        <inertial>
-            <!-- mass measured on average over four wooden sticks -->
+        <!-- mass measured on average over four wooden sticks -->
+        <inertial>
             <mass value="0.056" />
             <!-- ./cylinder_inertia.py 0.056 0.012 0.026 -->
@@ -260,7 +260,7 @@
             </geometry>
         </collision>
+        <!-- mass based on filament estimate from Prusa Slicer -->
         <inertial>
             <origin rpy="0 1.5707963267948966 0" xyz="0.03 0 0" />
-            <!-- mass based on filament estimate from Prusa Slicer -->
             <mass value="0.09874" />
             <!-- ./cylinder_inertia.py 0.09874 0.05 0.06 -->
@@ -281,7 +281,7 @@
             </geometry>
         </collision>
-        <inertial>
-            <origin rpy="0 0 0" xyz="0 0 0.015" />
-            <!-- mass guessed from spec -->
+        <!-- mass guessed from spec -->
+        <inertial>
+            <origin rpy="0 0 0" xyz="0 0 0.015" />
             <mass value="0.47" />
             <!-- ./cylinder_inertia.py 0.470 0.05 0.03 -->
@@ -315,7 +315,7 @@
             </geometry>
         </collision>
+        <!-- mass guessed from spec -->
         <inertial>
             <origin rpy="0 0 0" xyz="0 0 -0.0025" />
-            <!-- mass guessed from spec -->
             <mass value="0.015" />
             <!-- ./cylinder_inertia.py 0.015 0.023 0.005 -->
@@ -336,7 +336,7 @@
             </geometry>
         </collision>
+        <!-- mass measured with screws -->
         <inertial>
             <origin rpy="0 1.5707963267948966 0" xyz="0 0 0.025" />
-            <!-- mass measured with screws -->
             <mass value="0.05267" />
             <!-- ./cylinder_inertia.py 0.05267 0.025 0.09 -->
@@ -363,6 +363,6 @@
             <material name="light_wood" />
         </collision>
-        <inertial>
-            <!-- mass measured on average over four wooden sticks -->
+        <!-- mass measured on average over four wooden sticks -->
+        <inertial>
             <mass value="0.056" />
             <!-- ./cylinder_inertia.py 0.056 0.012 0.026 -->
@@ -389,7 +389,7 @@
             </geometry>
         </collision>
+        <!-- mass measured with screws -->
         <inertial>
             <origin rpy="0 0 0" xyz="0 0.002 0.0275" />
-            <!-- mass measured with screws -->
             <mass value="0.07863" />
             <!-- ./box_inertia.py 0.07863 0.092 0.068 0.056 -->
@@ -414,6 +414,6 @@
             </geometry>
         </collision>
-        <inertial>
-            <!-- mass is a pure guess (^_^") -->
+        <!-- mass is a pure guess (^_^") -->
+        <inertial>
             <mass value="0.02" />
             <!-- ./box_inertia.py 0.02 0.09 0.046 0.004 -->
@@ -439,7 +439,7 @@
             </geometry>
         </collision>
+        <!-- mass measured was 242.1 [g], minus 20 [g] for the plate, minus 50 [g] for the rotor -->
         <inertial>
             <origin rpy="0 0 0" xyz="0 0 0.01" />
-            <!-- mass measured was 242.1 [g], minus 20 [g] for the plate, minus 50 [g] for the rotor -->
             <mass value="0.1721" />
             <!-- ./cylinder_inertia.py 0.1721 0.03 0.018 -->
@@ -479,7 +479,7 @@
             </geometry>
         </collision>
-        <inertial>
-            <origin rpy="0 0 0" xyz="0 0 0.015" />
-            <!-- mass is a pure guess -->
+        <!-- mass is a pure guess -->
+        <inertial>
+            <origin rpy="0 0 0" xyz="0 0 0.015" />
             <mass value="0.05" />
             <!-- ./cylinder_inertia.py 0.05 0.034 0.016 -->
@@ -509,7 +509,7 @@
             </geometry>
         </collision>
+        <!-- mass measured with hub adapter -->
         <inertial>
             <origin rpy="0 0 0" xyz="0 0 0.0125" />
-            <!-- mass measured with hub adapter -->
             <mass value="0.0454" />
             <!-- ./cylinder_inertia.py 0.0454 0.039 0.025 -->
@@ -534,6 +534,6 @@
             </geometry>
         </collision>
-        <inertial>
-            <!-- mass measured on a real robot -->
+        <!-- mass measured on a real robot -->
+        <inertial>
             <mass value="0.08715" />
             <!-- ./cylinder_inertia.py 0.08715 0.05 0.04 -->
@@ -597,7 +597,7 @@
             </geometry>
         </collision>
-        <inertial>
-            <origin rpy="0 0 0" xyz="0 0 0.015" />
-            <!-- mass guessed from spec -->
+        <!-- mass guessed from spec -->
+        <inertial>
+            <origin rpy="0 0 0" xyz="0 0 0.015" />
             <mass value="0.47" />
             <!-- ./cylinder_inertia.py 0.470 0.05 0.03 -->
@@ -623,7 +623,7 @@
             </geometry>
         </collision>
+        <!-- mass guessed from spec -->
         <inertial>
             <origin rpy="0 0 0" xyz="0 0 -0.0025" />
-            <!-- mass guessed from spec -->
             <mass value="0.015" />
             <!-- ./cylinder_inertia.py 0.015 0.023 0.005 -->
@@ -652,7 +652,7 @@
             </geometry>
         </collision>
+        <!-- mass measured with screws -->
         <inertial>
             <origin rpy="0 1.5707963267948966 0" xyz="0 0 0.025" />
-            <!-- mass measured with screws -->
             <mass value="0.05267" />
             <!-- ./cylinder_inertia.py 0.05267 0.025 0.09 -->
@@ -679,6 +679,6 @@
             <material name="light_wood" />
         </collision>
-        <inertial>
-            <!-- mass measured on average over four wooden sticks -->
+        <!-- mass measured on average over four wooden sticks -->
+        <inertial>
             <mass value="0.056" />
             <!-- ./cylinder_inertia.py 0.056 0.012 0.026 -->
@@ -710,7 +710,7 @@
             </geometry>
         </collision>
+        <!-- mass based on filament estimate from Prusa Slicer -->
         <inertial>
             <origin rpy="0 1.5707963267948966 0" xyz="0.03 0 0" />
-            <!-- mass based on filament estimate from Prusa Slicer -->
             <mass value="0.09874" />
             <!-- ./cylinder_inertia.py 0.09874 0.05 0.06 -->
@@ -731,7 +731,7 @@
             </geometry>
         </collision>
-        <inertial>
-            <origin rpy="0 0 0" xyz="0 0 0.015" />
-            <!-- mass guessed from spec -->
+        <!-- mass guessed from spec -->
+        <inertial>
+            <origin rpy="0 0 0" xyz="0 0 0.015" />
             <mass value="0.47" />
             <!-- ./cylinder_inertia.py 0.470 0.05 0.03 -->
@@ -765,7 +765,7 @@
             </geometry>
         </collision>
+        <!-- mass guessed from spec -->
         <inertial>
             <origin rpy="0 0 0" xyz="0 0 -0.0025" />
-            <!-- mass guessed from spec -->
             <mass value="0.015" />
             <!-- ./cylinder_inertia.py 0.015 0.023 0.005 -->
@@ -786,7 +786,7 @@
             </geometry>
         </collision>
+        <!-- mass measured with screws -->
         <inertial>
             <origin rpy="0 1.5707963267948966 0" xyz="0 0 0.025" />
-            <!-- mass measured with screws -->
             <mass value="0.05267" />
             <!-- ./cylinder_inertia.py 0.05267 0.025 0.09 -->
@@ -813,6 +813,6 @@
             <material name="light_wood" />
         </collision>
-        <inertial>
-            <!-- mass measured on average over four wooden sticks -->
+        <!-- mass measured on average over four wooden sticks -->
+        <inertial>
             <mass value="0.056" />
             <!-- ./cylinder_inertia.py 0.056 0.012 0.026 -->
@@ -839,7 +839,7 @@
             </geometry>
         </collision>
+        <!-- mass measured with screws -->
         <inertial>
             <origin rpy="0 0 0" xyz="0 0.002 0.0275" />
-            <!-- mass measured with screws -->
             <mass value="0.07863" />
             <!-- ./box_inertia.py 0.07863 0.092 0.068 0.056 -->
@@ -864,6 +864,6 @@
             </geometry>
         </collision>
-        <inertial>
-            <!-- mass is a pure guess (^_^") -->
+        <!-- mass is a pure guess (^_^") -->
+        <inertial>
             <mass value="0.02" />
             <!-- ./box_inertia.py 0.02 0.09 0.046 0.004 -->
@@ -889,7 +889,7 @@
             </geometry>
         </collision>
+        <!-- mass measured was 242.1 [g], minus 20 [g] for the plate, minus 50 [g] for the rotor -->
         <inertial>
             <origin rpy="0 0 0" xyz="0 0 0.01" />
-            <!-- mass measured was 242.1 [g], minus 20 [g] for the plate, minus 50 [g] for the rotor -->
             <mass value="0.1721" />
             <!-- ./cylinder_inertia.py 0.1721 0.03 0.018 -->
@@ -929,7 +929,7 @@
             </geometry>
         </collision>
-        <inertial>
-            <origin rpy="0 0 0" xyz="0 0 0.015" />
-            <!-- mass is a pure guess -->
+        <!-- mass is a pure guess -->
+        <inertial>
+            <origin rpy="0 0 0" xyz="0 0 0.015" />
             <mass value="0.05" />
             <!-- ./cylinder_inertia.py 0.05 0.034 0.016 -->
@@ -959,7 +959,7 @@
             </geometry>
         </collision>
+        <!-- mass measured with hub adapter -->
         <inertial>
             <origin rpy="0 0 0" xyz="0 0 0.0125" />
-            <!-- mass measured with hub adapter -->
             <mass value="0.0454" />
             <!-- ./cylinder_inertia.py 0.0454 0.039 0.025 -->
@@ -984,6 +984,6 @@
             </geometry>
         </collision>
-        <inertial>
-            <!-- mass measured on a real tire -->
+        <!-- mass measured on a real tire -->
+        <inertial>
             <mass value="0.08715" />
             <!-- ./cylinder_inertia.py 0.08715 0.05 0.04 -->

Commit message: WIP: Another box inertia

File: xacro/upkie.xacro (robot description, xacro)
@@ -94,9 +94,5 @@
         </collision>
         <!-- mass measurement was imprecise -->
-        <inertial>
-            <mass value="0.8" />
-            <!-- ./box_inertia.py 0.800 0.13 0.074 0.055 -->
-            <inertia ixx="0.0005667333333333332" ixy="0" ixz="0" iyx="0" iyy="0.0013283333333333335" iyz="0" izx="0" izy="0" izz="0.0014917333333333332" />
-        </inertial>
+        <xacro:box_inertia mass="0.8" len_x="0.13" len_y="0.074" len_z="0.055" />
     </link>
     <joint name="battery_fix" type="fixed">

Commit message: WIP: Box inertia with shifted origin

File: xacro/upkie.xacro (robot description, xacro)
@@ -122,10 +122,8 @@
         </collision>
         <!-- mass measured on a real robot -->
-        <inertial>
-            <origin rpy="0 0 0" xyz="0 0 0.01" />
-            <mass value="0.0525" />
-            <!-- ./box_inertia.py 0.0525 0.120 0.07 0.04 -->
-            <inertia ixx="2.84375e-05" ixy="0" ixz="0" iyx="0" iyy="7e-05" iyz="0" izx="0" izy="0" izz="8.44375e-05" />
-        </inertial>
+        <xacro:box_inertia
+            rpy="0 0 0" xyz="0 0 0.01"
+            mass="0.0525"
+            len_x="0.120" len_y="0.07" len_z="0.04" />
     </link>
     <joint name="handle_fix" type="fixed">

Commit message: Replace all remaining box inertias by xacro macros

File: xacro/upkie.xacro (robot description, xacro)
@@ -390,10 +390,8 @@
         </collision>
         <!-- mass measured with screws -->
-        <inertial>
-            <origin rpy="0 0 0" xyz="0 0.002 0.0275" />
-            <mass value="0.07863" />
-            <!-- ./box_inertia.py 0.07863 0.092 0.068 0.056 -->
-            <inertia ixx="5.084740000000001e-05" ixy="0" ixz="0" iyx="0" iyy="7.6009e-05" iyz="0" izx="0" izy="0" izz="8.575912e-05" />
-        </inertial>
+        <xacro:box_inertia
+            rpy="0 0 0" xyz="0 0.002 0.0275"
+            mass="0.07863"
+            len_x="0.092" len_y="0.068" len_z="0.056" />
     </link>
     <joint name="left_ankle_base_fix" type="fixed">
@@ -415,9 +413,8 @@
         </collision>
         <!-- mass is a pure guess (^_^") -->
-        <inertial>
-            <mass value="0.02" />
-            <!-- ./box_inertia.py 0.02 0.09 0.046 0.004 -->
-            <inertia ixx="3.5533333333333333e-06" ixy="0" ixz="0" iyx="0" iyy="1.3526666666666667e-05" iyz="0" izx="0" izy="0" izz="1.7026666666666667e-05" />
-        </inertial>
+        <xacro:box_inertia
+            rpy="0 0 0" xyz="0 0 0"
+            mass="0.02"
+            len_x="0.09" len_y="0.046" len_z="0.004" />
     </link>
     <joint name="left_ankle_plate_fix" type="fixed">
@@ -840,10 +837,8 @@
         </collision>
         <!-- mass measured with screws -->
-        <inertial>
-            <origin rpy="0 0 0" xyz="0 0.002 0.0275" />
-            <mass value="0.07863" />
-            <!-- ./box_inertia.py 0.07863 0.092 0.068 0.056 -->
-            <inertia ixx="5.084740000000001e-05" ixy="0" ixz="0" iyx="0" iyy="7.6009e-05" iyz="0" izx="0" izy="0" izz="8.575912e-05" />
-        </inertial>
+        <xacro:box_inertia
+            rpy="0 0 0" xyz="0 0.002 0.0275"
+            mass="0.07863"
+            len_x="0.092" len_y="0.068" len_z="0.056" />
     </link>
     <joint name="right_ankle_base_fix" type="fixed">
@@ -865,9 +860,8 @@
         </collision>
         <!-- mass is a pure guess (^_^") -->
-        <inertial>
-            <mass value="0.02" />
-            <!-- ./box_inertia.py 0.02 0.09 0.046 0.004 -->
-            <inertia ixx="3.5533333333333333e-06" ixy="0" ixz="0" iyx="0" iyy="1.3526666666666667e-05" iyz="0" izx="0" izy="0" izz="1.7026666666666667e-05" />
-        </inertial>
+        <xacro:box_inertia
+            rpy="0 0 0" xyz="0 0 0"
+            mass="0.02"
+            len_x="0.09" len_y="0.046" len_z="0.004" />
     </link>
     <joint name="right_ankle_plate_fix" type="fixed">

Commit message: WIP: Compute cylinder inertias via xacro

File: xacro/upkie.xacro (robot description, xacro)
@@ -7,4 +7,5 @@
 <robot name="upkie" xmlns:xacro="http://ros.org/wiki/xacro">
     <xacro:include filename="xacro/box_inertia.xacro" />
+    <xacro:include filename="xacro/cylinder_inertia.xacro" />
     <material name="black">
         <color rgba="0.1 0.1 0.1 1" />
@@ -148,10 +149,8 @@
         </collision>
         <!-- mass guessed from spec -->
-        <inertial>
-            <origin rpy="0 0 0" xyz="0 0 0.015" />
-            <mass value="0.47" />
-            <!-- ./cylinder_inertia.py 0.470 0.05 0.03 -->
-            <inertia ixx="0.000329" ixy="0" ixz="0" iyx="0" iyy="0.000329" iyz="0" izx="0" izy="0" izz="0.0005875" />
-        </inertial>
+        <xacro:cylinder_inertia
+            rpy="0 0 0" xyz="0 0 0.015"
+            mass="0.47"
+            radius="0.05" length="0.03" />
     </link>
     <joint name="left_hip_qdd100_stator_fix" type="fixed">

Commit message: WIP: Update cylinder inertias

File: xacro/upkie.xacro (robot description, xacro)
@@ -173,10 +173,8 @@
         </collision>
         <!-- mass guessed from spec -->
-        <inertial>
-            <origin rpy="0 0 0" xyz="0 0 -0.0025" />
-            <mass value="0.015" />
-            <!-- ./cylinder_inertia.py 0.015 0.023 0.005 -->
-            <inertia ixx="2.0149999999999998e-06" ixy="0" ixz="0" iyx="0" iyy="2.0149999999999998e-06" iyz="0" izx="0" izy="0" izz="3.9675e-06" />
-        </inertial>
+        <xacro:cylinder_inertia
+            rpy="0 0 0" xyz="0 0 -0.0025"
+            mass="0.015"
+            radius="0.023" length="0.005" />
     </link>
     <joint name="left_hip" type="revolute">
@@ -202,10 +200,8 @@
         </collision>
         <!-- mass measured with screws -->
-        <inertial>
-            <origin rpy="0 1.5707963267948966 0" xyz="0 0 0.025" />
-            <mass value="0.05267" />
-            <!-- ./cylinder_inertia.py 0.05267 0.025 0.09 -->
-            <inertia ixx="4.37819375e-05" ixy="0" ixz="0" iyx="0" iyy="4.37819375e-05" iyz="0" izx="0" izy="0" izz="1.6459375e-05" />
-        </inertial>
+        <xacro:cylinder_inertia
+            rpy="0 1.5707963267948966 0" xyz="0 0 0.025"
+            mass="0.05267"
+            radius="0.025" length="0.09" />
     </link>
     <joint name="left_hip_horn_fix" type="fixed">
@@ -229,9 +225,8 @@
         </collision>
         <!-- mass measured on average over four wooden sticks -->
-        <inertial>
-            <mass value="0.056" />
-            <!-- ./cylinder_inertia.py 0.056 0.012 0.026 -->
-            <inertia ixx="5.170666666666667e-06" ixy="0" ixz="0" iyx="0" iyy="5.170666666666667e-06" iyz="0" izx="0" izy="0" izz="4.0320000000000005e-06" />
-        </inertial>
+        <xacro:cylinder_inertia
+            rpy="0 0 0" xyz="0 0 0"
+            mass="0.056"
+            radius="0.012" length="0.026" />
     </link>
     <joint name="left_femur_fix" type="fixed">
@@ -260,10 +255,8 @@
         </collision>
         <!-- mass based on filament estimate from Prusa Slicer -->
-        <inertial>
-            <origin rpy="0 1.5707963267948966 0" xyz="0.03 0 0" />
-            <mass value="0.09874" />
-            <!-- ./cylinder_inertia.py 0.09874 0.05 0.06 -->
-            <inertia ixx="9.133450000000001e-05" ixy="0" ixz="0" iyx="0" iyy="9.133450000000001e-05" iyz="0" izx="0" izy="0" izz="0.000123425" />
-        </inertial>
+        <xacro:cylinder_inertia
+            rpy="0 1.5707963267948966 0" xyz="0.03 0 0"
+            mass="0.09874"
+            radius="0.05" length="0.06" />
     </link>
     <link name="left_knee_qdd100_stator">
@@ -281,10 +274,8 @@
         </collision>
         <!-- mass guessed from spec -->
-        <inertial>
-            <origin rpy="0 0 0" xyz="0 0 0.015" />
-            <mass value="0.47" />
-            <!-- ./cylinder_inertia.py 0.470 0.05 0.03 -->
-            <inertia ixx="0.000329" ixy="0" ixz="0" iyx="0" iyy="0.000329" iyz="0" izx="0" izy="0" izz="0.0005875" />
-        </inertial>
+        <xacro:cylinder_inertia
+            rpy="0 0 0" xyz="0 0 0.015"
+            mass="0.47"
+            radius="0.05" length="0.03" />
     </link>
     <joint name="left_knee_qdd100_stator_fix" type="fixed">
@@ -315,10 +306,8 @@
         </collision>
         <!-- mass guessed from spec -->
-        <inertial>
-            <origin rpy="0 0 0" xyz="0 0 -0.0025" />
-            <mass value="0.015" />
-            <!-- ./cylinder_inertia.py 0.015 0.023 0.005 -->
-            <inertia ixx="2.0149999999999998e-06" ixy="0" ixz="0" iyx="0" iyy="2.0149999999999998e-06" iyz="0" izx="0" izy="0" izz="3.9675e-06" />
-        </inertial>
+        <xacro:cylinder_inertia
+            rpy="0 0 0" xyz="0 0 -0.0025"
+            mass="0.015"
+            radius="0.023" length="0.005" />
     </link>
     <link name="left_knee_horn">
@@ -336,10 +325,8 @@
         </collision>
         <!-- mass measured with screws -->
-        <inertial>
-            <origin rpy="0 1.5707963267948966 0" xyz="0 0 0.025" />
-            <mass value="0.05267" />
-            <!-- ./cylinder_inertia.py 0.05267 0.025 0.09 -->
-            <inertia ixx="4.37819375e-05" ixy="0" ixz="0" iyx="0" iyy="4.37819375e-05" iyz="0" izx="0" izy="0" izz="1.6459375e-05" />
-        </inertial>
+        <xacro:cylinder_inertia
+            rpy="0 1.5707963267948966 0" xyz="0 0 0.025"
+            mass="0.05267"
+            radius="0.025" length="0.09" />
     </link>
     <joint name="left_knee_horn_fix" type="fixed">
