Commit message: WIP: Update cylinder inertias

File: xacro/upkie.xacro (robot description, xacro)
@@ -350,9 +350,8 @@
         </collision>
         <!-- mass measured on average over four wooden sticks -->
-        <inertial>
-            <mass value="0.056" />
-            <!-- ./cylinder_inertia.py 0.056 0.012 0.026 -->
-            <inertia ixx="5.170666666666667e-06" ixy="0" ixz="0" iyx="0" iyy="5.170666666666667e-06" iyz="0" izx="0" izy="0" izz="4.0320000000000005e-06" />
-        </inertial>
+        <xacro:cylinder_inertia
+            rpy="0 0 0" xyz="0 0 0"
+            mass="0.056"
+            radius="0.012" length="0.026" />
     </link>
     <joint name="left_tibia_fix" type="fixed">
@@ -663,9 +662,8 @@
         </collision>
         <!-- mass measured on average over four wooden sticks -->
-        <inertial>
-            <mass value="0.056" />
-            <!-- ./cylinder_inertia.py 0.056 0.012 0.026 -->
-            <inertia ixx="5.170666666666667e-06" ixy="0" ixz="0" iyx="0" iyy="5.170666666666667e-06" iyz="0" izx="0" izy="0" izz="4.0320000000000005e-06" />
-        </inertial>
+        <xacro:cylinder_inertia
+            rpy="0 0 0" xyz="0 0 0"
+            mass="0.056"
+            radius="0.012" length="0.026" />
     </link>
     <joint name="right_femur_fix" type="fixed">
@@ -797,9 +795,8 @@
         </collision>
         <!-- mass measured on average over four wooden sticks -->
-        <inertial>
-            <mass value="0.056" />
-            <!-- ./cylinder_inertia.py 0.056 0.012 0.026 -->
-            <inertia ixx="5.170666666666667e-06" ixy="0" ixz="0" iyx="0" iyy="5.170666666666667e-06" iyz="0" izx="0" izy="0" izz="4.0320000000000005e-06" />
-        </inertial>
+        <xacro:cylinder_inertia
+            rpy="0 0 0" xyz="0 0 0"
+            mass="0.056"
+            radius="0.012" length="0.026" />
     </link>
     <joint name="right_tibia_fix" type="fixed">
@@ -870,10 +867,8 @@
         </collision>
         <!-- mass measured was 242.1 [g], minus 20 [g] for the plate, minus 50 [g] for the rotor -->
-        <inertial>
-            <origin rpy="0 0 0" xyz="0 0 0.01" />
-            <mass value="0.1721" />
-            <!-- ./cylinder_inertia.py 0.1721 0.03 0.018 -->
-            <inertia ixx="4.3369200000000005e-05" ixy="0" ixz="0" iyx="0" iyy="4.3369200000000005e-05" iyz="0" izx="0" izy="0" izz="7.7445e-05" />
-        </inertial>
+        <xacro:cylinder_inertia
+            rpy="0 0 0" xyz="0 0 0.01"
+            mass="0.1721"
+            radius="0.03" length="0.018" />
     </link>
     <joint name="right_ankle_mj5208_stator_fix" type="fixed">
@@ -910,10 +905,8 @@
         </collision>
         <!-- mass is a pure guess -->
-        <inertial>
-            <origin rpy="0 0 0" xyz="0 0 0.015" />
-            <mass value="0.05" />
-            <!-- ./cylinder_inertia.py 0.05 0.034 0.016 -->
-            <inertia ixx="1.551666666666667e-05" ixy="0" ixz="0" iyx="0" iyy="1.551666666666667e-05" iyz="0" izx="0" izy="0" izz="2.8900000000000005e-05" />
-        </inertial>
+        <xacro:cylinder_inertia
+            rpy="0 0 0" xyz="0 0 0.015"
+            mass="0.05"
+            radius="0.034" length="0.016" />
     </link>
     <joint name="right_wheel" type="revolute">

Commit message: WIP: Update more cylinder inertias

File: xacro/upkie.xacro (robot description, xacro)
@@ -422,10 +422,8 @@
         </collision>
         <!-- mass measured was 242.1 [g], minus 20 [g] for the plate, minus 50 [g] for the rotor -->
-        <inertial>
-            <origin rpy="0 0 0" xyz="0 0 0.01" />
-            <mass value="0.1721" />
-            <!-- ./cylinder_inertia.py 0.1721 0.03 0.018 -->
-            <inertia ixx="4.3369200000000005e-05" ixy="0" ixz="0" iyx="0" iyy="4.3369200000000005e-05" iyz="0" izx="0" izy="0" izz="7.7445e-05" />
-        </inertial>
+        <xacro:cylinder_inertia
+            rpy="0 0 0" xyz="0 0 0.01"
+            mass="0.1721"
+            radius="0.03" length="0.018" />
     </link>
     <joint name="left_ankle_mj5208_stator_fix" type="fixed">
@@ -462,10 +460,8 @@
         </collision>
         <!-- mass is a pure guess -->
-        <inertial>
-            <origin rpy="0 0 0" xyz="0 0 0.015" />
-            <mass value="0.05" />
-            <!-- ./cylinder_inertia.py 0.05 0.034 0.016 -->
-            <inertia ixx="1.551666666666667e-05" ixy="0" ixz="0" iyx="0" iyy="1.551666666666667e-05" iyz="0" izx="0" izy="0" izz="2.8900000000000005e-05" />
-        </inertial>
+        <xacro:cylinder_inertia
+            rpy="0 0 0" xyz="0 0 0.015"
+            mass="0.05"
+            radius="0.034" length="0.016" />
     </link>
     <joint name="left_wheel" type="revolute">
@@ -492,10 +488,8 @@
         </collision>
         <!-- mass measured with hub adapter -->
-        <inertial>
-            <origin rpy="0 0 0" xyz="0 0 0.0125" />
-            <mass value="0.0454" />
-            <!-- ./cylinder_inertia.py 0.0454 0.039 0.025 -->
-            <inertia ixx="1.9627933333333332e-05" ixy="0" ixz="0" iyx="0" iyy="1.9627933333333332e-05" iyz="0" izx="0" izy="0" izz="3.45267e-05" />
-        </inertial>
+        <xacro:cylinder_inertia
+            rpy="0 0 0" xyz="0 0 0.0125"
+            mass="0.0454"
+            radius="0.039" length="0.025" />
     </link>
     <joint name="left_wheel_hub_fix" type="fixed">
@@ -933,10 +927,8 @@
         </collision>
         <!-- mass measured with hub adapter -->
-        <inertial>
-            <origin rpy="0 0 0" xyz="0 0 0.0125" />
-            <mass value="0.0454" />
-            <!-- ./cylinder_inertia.py 0.0454 0.039 0.025 -->
-            <inertia ixx="1.9627933333333332e-05" ixy="0" ixz="0" iyx="0" iyy="1.9627933333333332e-05" iyz="0" izx="0" izy="0" izz="3.45267e-05" />
-        </inertial>
+        <xacro:cylinder_inertia
+            rpy="0 0 0" xyz="0 0 0.0125"
+            mass="0.0454"
+            radius="0.039" length="0.025" />
     </link>
     <joint name="right_wheel_hub_fix" type="fixed">
@@ -958,9 +950,8 @@
         </collision>
         <!-- mass measured on a real tire -->
-        <inertial>
-            <mass value="0.08715" />
-            <!-- ./cylinder_inertia.py 0.08715 0.05 0.04 -->
-            <inertia ixx="6.608875000000002e-05" ixy="0" ixz="0" iyx="0" iyy="6.608875000000002e-05" iyz="0" izx="0" izy="0" izz="0.00010893750000000003" />
-        </inertial>
+        <xacro:cylinder_inertia
+            rpy="0 0 0" xyz="0 0 0"
+            mass="0.08715"
+            radius="0.05" length="0.04" />
         <contact>
             <lateral_friction value="1.0" />

Commit message: WIP: Woah, this is penible...

File: xacro/upkie.xacro (robot description, xacro)
@@ -511,443 +511,4 @@
         </collision>
         <!-- mass measured on a real robot -->
-        <inertial>
-            <mass value="0.08715" />
-            <!-- ./cylinder_inertia.py 0.08715 0.05 0.04 -->
-            <inertia ixx="6.608875000000002e-05" ixy="0" ixz="0" iyx="0" iyy="6.608875000000002e-05" iyz="0" izx="0" izy="0" izz="0.00010893750000000003" />
-        </inertial>
-        <contact>
-            <lateral_friction value="1.0" />
-            <rolling_friction value="0.01" />
-            <stiffness value="30000" />
-            <damping value="1000" />
-        </contact>
-    </link>
-    <joint name="left_wheel_fix" type="fixed">
-        <parent link="left_wheel_hub" />
-        <child link="left_wheel_tire" />
-        <origin rpy="0 0 0" xyz="0 0 0.0209" />
-    </joint>
-    <link name="left_contact">
-        <!-- virtual link -->
-        <inertial>
-            <!-- mass should not be zero [1] -->
-            <mass value="0.001" />
-            <origin rpy="0 0 0" xyz="0 0 0" />
-            <inertia ixx="0" ixy="0" ixz="0" iyy="0" iyz="0" izz="0" />
-        </inertial>
-    </link>
-    <joint name="left_contact_fix" type="fixed">
-        <parent link="left_wheel_tire" />
-        <child link="left_contact" />
-        <!-- contact target is a bit inside to avoid collisions with its box -->
-        <!-- tangent contact surface would be xyz="0 0.05 0" -->
-        <origin rpy="1.5707963267948966 0 0" xyz="0 0.047 0" />
-    </joint>
-    <link name="left_wheel_center">
-        <!-- virtual link -->
-        <inertial>
-            <!-- mass should not be zero [1] -->
-            <mass value="0.001" />
-            <origin rpy="0 0 0" xyz="0 0 0" />
-            <inertia ixx="0" ixy="0" ixz="0" iyy="0" iyz="0" izz="0" />
-        </inertial>
-    </link>
-    <joint name="left_wheel_center_fix" type="fixed">
-        <parent link="left_wheel_tire" />
-        <child link="left_wheel_center" />
-        <origin rpy="1.5707963267948966 3.141592653589793 0" xyz="0 0 0" />
-    </joint>
-    <!-- Right leg -->
-    <!-- Right hip -->
-    <link name="right_hip_qdd100_stator">
-        <visual>
-            <geometry>
-                <mesh filename="package://upkie_description/meshes/mjbots/qdd100_stator.stl" />
-            </geometry>
-            <material name="black" />
-        </visual>
-        <collision>
-            <origin rpy="0 0 0" xyz="0 0 0.015" />
-            <geometry>
-                <cylinder length="0.03" radius="0.05" />
-            </geometry>
-        </collision>
-        <!-- mass guessed from spec -->
-        <inertial>
-            <origin rpy="0 0 0" xyz="0 0 0.015" />
-            <mass value="0.47" />
-            <!-- ./cylinder_inertia.py 0.470 0.05 0.03 -->
-            <inertia ixx="0.000329" ixy="0" ixz="0" iyx="0" iyy="0.000329" iyz="0" izx="0" izy="0" izz="0.0005875" />
-        </inertial>
-    </link>
-    <joint name="right_hip_qdd100_stator_fix" type="fixed">
-        <origin rpy="1.5707963267948966 3.141592653589793 0" xyz="0.0 -0.085 -0.064" />
-        <parent link="torso" />
-        <child link="right_hip_qdd100_stator" />
-    </joint>
-    <link name="right_hip_qdd100_rotor">
-        <visual>
-            <geometry>
-                <mesh filename="package://upkie_description/meshes/mjbots/qdd100_rotor.stl" />
-            </geometry>
-            <material name="black" />
-        </visual>
-        <collision>
-            <origin rpy="0 0 0" xyz="0 0 -0.0025" />
-            <geometry>
-                <cylinder length="0.005" radius="0.023" />
-            </geometry>
-        </collision>
-        <!-- mass guessed from spec -->
-        <inertial>
-            <origin rpy="0 0 0" xyz="0 0 -0.0025" />
-            <mass value="0.015" />
-            <!-- ./cylinder_inertia.py 0.015 0.023 0.005 -->
-            <inertia ixx="2.0149999999999998e-06" ixy="0" ixz="0" iyx="0" iyy="2.0149999999999998e-06" iyz="0" izx="0" izy="0" izz="3.9675e-06" />
-        </inertial>
-    </link>
-    <joint name="right_hip" type="revolute">
-        <parent link="right_hip_qdd100_stator" />
-        <child link="right_hip_qdd100_rotor" />
-        <origin rpy="0 0 0" xyz="0 0 0.0292" />
-        <!-- negative z-axis: search "moteus-direction-configuration" -->
-        <axis xyz="0 0 -1" />
-        <limit effort="16.0" lower="-1.26" upper="1.26" velocity="28.8" />
-    </joint>
-    <link name="right_hip_horn">
-        <visual>
-            <geometry>
-                <mesh filename="package://upkie_description/meshes/mjbots/qdd100_horn.stl" />
-            </geometry>
-            <material name="black" />
-        </visual>
-        <collision>
-            <origin rpy="0 1.5707963267948966 0" xyz="0 0 0.025" />
-            <geometry>
-                <cylinder length="0.09" radius="0.025" />
-            </geometry>
-        </collision>
-        <!-- mass measured with screws -->
-        <inertial>
-            <origin rpy="0 1.5707963267948966 0" xyz="0 0 0.025" />
-            <mass value="0.05267" />
-            <!-- ./cylinder_inertia.py 0.05267 0.025 0.09 -->
-            <inertia ixx="4.37819375e-05" ixy="0" ixz="0" iyx="0" iyy="4.37819375e-05" iyz="0" izx="0" izy="0" izz="1.6459375e-05" />
-        </inertial>
-    </link>
-    <joint name="right_hip_horn_fix" type="fixed">
-        <parent link="right_hip_qdd100_rotor" />
-        <child link="right_hip_horn" />
-        <origin rpy="0 0 1.5707963267948966" xyz="0 0 0" />
-    </joint>
-    <!-- Right femur -->
-    <link name="right_femur">
-        <visual>
-            <geometry>
-                <cylinder length="0.25" radius="0.011" />
-            </geometry>
-            <material name="light_wood" />
-        </visual>
-        <collision>
-            <geometry>
-                <cylinder length="0.26" radius="0.012" />
-            </geometry>
-            <material name="light_wood" />
-        </collision>
-        <!-- mass measured on average over four wooden sticks -->
-        <xacro:cylinder_inertia
-            rpy="0 0 0" xyz="0 0 0"
-            mass="0.056"
-            radius="0.012" length="0.026" />
-    </link>
-    <joint name="right_femur_fix" type="fixed">
-        <parent link="right_hip_qdd100_rotor" />
-        <child link="right_femur" />
-        <origin rpy="1.5707963267948966 0 0" xyz="0 0.07 0.025" />
-    </joint>
-    <!-- Right knee -->
-    <joint name="right_knee_stator_fix" type="fixed">
-        <parent link="right_femur" />
-        <child link="right_knee_stator" />
-        <origin rpy="0 0 -1.5707963267948966" xyz="0 0.042 -0.098" />
-    </joint>
-    <link name="right_knee_stator">
-        <visual>
-            <geometry>
-                <mesh filename="package://upkie_description/meshes/knee_stator.stl" />
-            </geometry>
-            <material name="terracotta_light" />
-        </visual>
-        <collision>
-            <origin rpy="0 1.5707963267948966 0" xyz="0.03 0 0" />
-            <geometry>
-                <cylinder length="0.06" radius="0.05" />
-            </geometry>
-        </collision>
-        <!-- mass based on filament estimate from Prusa Slicer -->
-        <inertial>
-            <origin rpy="0 1.5707963267948966 0" xyz="0.03 0 0" />
-            <mass value="0.09874" />
-            <!-- ./cylinder_inertia.py 0.09874 0.05 0.06 -->
-            <inertia ixx="9.133450000000001e-05" ixy="0" ixz="0" iyx="0" iyy="9.133450000000001e-05" iyz="0" izx="0" izy="0" izz="0.000123425" />
-        </inertial>
-    </link>
-    <link name="right_knee_qdd100_stator">
-        <visual>
-            <geometry>
-                <mesh filename="package://upkie_description/meshes/mjbots/qdd100_stator.stl" />
-            </geometry>
-            <material name="black" />
-        </visual>
-        <collision>
-            <origin rpy="0 0 0" xyz="0 0 0.015" />
-            <geometry>
-                <cylinder length="0.03" radius="0.05" />
-            </geometry>
-        </collision>
-        <!-- mass guessed from spec -->
-        <inertial>
-            <origin rpy="0 0 0" xyz="0 0 0.015" />
-            <mass value="0.47" />
-            <!-- ./cylinder_inertia.py 0.470 0.05 0.03 -->
-            <inertia ixx="0.000329" ixy="0" ixz="0" iyx="0" iyy="0.000329" iyz="0" izx="0" izy="0" izz="0.0005875" />
-        </inertial>
-    </link>
-    <joint name="right_knee_qdd100_stator_fix" type="fixed">
-        <parent link="right_knee_stator" />
-        <child link="right_knee_qdd100_stator" />
-        <origin rpy="-1.5707963267948966 0 1.5707963267948966" xyz="0 0 0" />
-    </joint>
-    <joint name="right_knee" type="revolute">
-        <parent link="right_knee_qdd100_stator" />
-        <child link="right_knee_qdd100_rotor" />
-        <origin rpy="0 0 0" xyz="0 0 0.0292" />
-        <!-- negative z-axis: search "moteus-direction-configuration" -->
-        <axis xyz="0 0 -1" />
-        <limit effort="16.0" lower="-2.51" upper="2.51" velocity="28.8" />
-    </joint>
-    <link name="right_knee_qdd100_rotor">
-        <visual>
-            <geometry>
-                <mesh filename="package://upkie_description/meshes/mjbots/qdd100_rotor.stl" />
-            </geometry>
-            <material name="black" />
-        </visual>
-        <collision>
-            <origin rpy="0 0 0" xyz="0 0 -0.0025" />
-            <geometry>
-                <cylinder length="0.005" radius="0.023" />
-            </geometry>
-        </collision>
-        <!-- mass guessed from spec -->
-        <inertial>
-            <origin rpy="0 0 0" xyz="0 0 -0.0025" />
-            <mass value="0.015" />
-            <!-- ./cylinder_inertia.py 0.015 0.023 0.005 -->
-            <inertia ixx="2.0149999999999998e-06" ixy="0" ixz="0" iyx="0" iyy="2.0149999999999998e-06" iyz="0" izx="0" izy="0" izz="3.9675e-06" />
-        </inertial>
-    </link>
-    <link name="right_knee_horn">
-        <visual>
-            <geometry>
-                <mesh filename="package://upkie_description/meshes/mjbots/qdd100_horn.stl" />
-            </geometry>
-            <material name="terracotta_light" />
-        </visual>
-        <collision>
-            <origin rpy="0 1.5707963267948966 0" xyz="0 0 0.025" />
-            <geometry>
-                <cylinder length="0.09" radius="0.025" />
-            </geometry>
-        </collision>
-        <!-- mass measured with screws -->
-        <inertial>
-            <origin rpy="0 1.5707963267948966 0" xyz="0 0 0.025" />
-            <mass value="0.05267" />
-            <!-- ./cylinder_inertia.py 0.05267 0.025 0.09 -->
-            <inertia ixx="4.37819375e-05" ixy="0" ixz="0" iyx="0" iyy="4.37819375e-05" iyz="0" izx="0" izy="0" izz="1.6459375e-05" />
-        </inertial>
-    </link>
-    <joint name="right_knee_horn_fix" type="fixed">
-        <parent link="right_knee_qdd100_rotor" />
-        <child link="right_knee_horn" />
-        <origin rpy="0 0 1.5707963267948966" xyz="0 0 0" />
-    </joint>
-    <!-- Right tibia -->
-    <link name="right_tibia">
-        <visual>
-            <geometry>
-                <cylinder length="0.25" radius="0.011" />
-            </geometry>
-            <material name="light_wood" />
-        </visual>
-        <collision>
-            <geometry>
-                <cylinder length="0.26" radius="0.012" />
-            </geometry>
-            <material name="light_wood" />
-        </collision>
-        <!-- mass measured on average over four wooden sticks -->
-        <xacro:cylinder_inertia
-            rpy="0 0 0" xyz="0 0 0"
-            mass="0.056"
-            radius="0.012" length="0.026" />
-    </link>
-    <joint name="right_tibia_fix" type="fixed">
-        <parent link="right_knee_qdd100_rotor" />
-        <child link="right_tibia" />
-        <origin rpy="1.5707963267948966 3.141592653589793 0" xyz="0 0.07 0.025" />
-    </joint>
-    <!-- Right ankle -->
-    <link name="right_ankle_base">
-        <visual>
-            <geometry>
-                <mesh filename="package://upkie_description/meshes/ankle_stator.stl" />
-            </geometry>
-            <material name="chalky_blue" />
-        </visual>
-        <collision>
-            <origin rpy="0 0 0" xyz="0 0.002 0.0275" />
-            <geometry>
-                <box size="0.092 0.068 0.056" />
-            </geometry>
-        </collision>
-        <!-- mass measured with screws -->
-        <xacro:box_inertia
-            rpy="0 0 0" xyz="0 0.002 0.0275"
-            mass="0.07863"
-            len_x="0.092" len_y="0.068" len_z="0.056" />
-    </link>
-    <joint name="right_ankle_base_fix" type="fixed">
-        <parent link="right_tibia" />
-        <child link="right_ankle_base" />
-        <origin rpy="1.5707963267948966 0 0" xyz="0 0.034 -0.105" />
-    </joint>
-    <link name="right_ankle_plate">
-        <visual>
-            <geometry>
-                <box size="0.08 0.045 0.003" />
-            </geometry>
-            <material name="light_gray" />
-        </visual>
-        <collision>
-            <geometry>
-                <box size="0.09 0.046 0.004" />
-            </geometry>
-        </collision>
-        <!-- mass is a pure guess (^_^") -->
-        <xacro:box_inertia
-            rpy="0 0 0" xyz="0 0 0"
-            mass="0.02"
-            len_x="0.09" len_y="0.046" len_z="0.004" />
-    </link>
-    <joint name="right_ankle_plate_fix" type="fixed">
-        <parent link="right_ankle_base" />
-        <child link="right_ankle_plate" />
-        <origin rpy="0 0 0" xyz="0 0 -0.0015" />
-    </joint>
-    <link name="right_ankle_mj5208_stator">
-        <visual>
-            <geometry>
-                <mesh filename="package://upkie_description/meshes/mjbots/mj5208_stator.stl" />
-            </geometry>
-            <material name="mj5208_stator" />
-        </visual>
-        <collision>
-            <origin rpy="0 0 0" xyz="0 0 0.01" />
-            <geometry>
-                <cylinder length="0.018" radius="0.03" />
-            </geometry>
-        </collision>
-        <!-- mass measured was 242.1 [g], minus 20 [g] for the plate, minus 50 [g] for the rotor -->
-        <xacro:cylinder_inertia
-            rpy="0 0 0" xyz="0 0 0.01"
-            mass="0.1721"
-            radius="0.03" length="0.018" />
-    </link>
-    <joint name="right_ankle_mj5208_stator_fix" type="fixed">
-        <parent link="right_ankle_plate" />
-        <child link="right_ankle_mj5208_stator" />
-        <origin rpy="3.141592653589793 0 0" xyz="0 0 -0.0015" />
-    </joint>
-    <link name="right_anchor">
-        <!-- virtual link -->
-        <inertial>
-            <!-- mass should not be zero [1] -->
-            <mass value="0.001" />
-            <origin rpy="0 0 0" xyz="0 0 0" />
-            <inertia ixx="0" ixy="0" ixz="0" iyy="0" iyz="0" izz="0" />
-        </inertial>
-    </link>
-    <joint name="right_anchor_fix" type="fixed">
-        <parent link="right_ankle_mj5208_stator" />
-        <child link="right_anchor" />
-        <origin rpy="1.5707963267948966 0 0" xyz="0 0.0545 0.048" />
-    </joint>
-    <link name="right_ankle_mj5208_rotor">
-        <visual>
-            <geometry>
-                <mesh filename="package://upkie_description/meshes/mjbots/mj5208_rotor.stl" />
-            </geometry>
-            <material name="mj5208_rotor" />
-        </visual>
-        <collision>
-            <origin rpy="0 0 0" xyz="0 0 0.015" />
-            <geometry>
-                <cylinder length="0.016" radius="0.034" />
-            </geometry>
-        </collision>
-        <!-- mass is a pure guess -->
-        <xacro:cylinder_inertia
-            rpy="0 0 0" xyz="0 0 0.015"
-            mass="0.05"
-            radius="0.034" length="0.016" />
-    </link>
-    <joint name="right_wheel" type="revolute">
-        <parent link="right_ankle_mj5208_stator" />
-        <child link="right_ankle_mj5208_rotor" />
-        <origin rpy="0 0 0" xyz="0 0 0" />
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