Commit message: Replace all remaining cylinder inertias

File: xacro/upkie.xacro (robot description, xacro)
@@ -597,10 +597,8 @@
         </collision>
         <!-- mass guessed from spec -->
-        <inertial>
-            <origin rpy="0 0 0" xyz="0 0 -0.0025" />
-            <mass value="0.015" />
-            <!-- ./cylinder_inertia.py 0.015 0.023 0.005 -->
-            <inertia ixx="2.0149999999999998e-06" ixy="0" ixz="0" iyx="0" iyy="2.0149999999999998e-06" iyz="0" izx="0" izy="0" izz="3.9675e-06" />
-        </inertial>
+        <xacro:cylinder_inertia
+            rpy="0 0 0" xyz="0 0 -0.0025"
+            mass="0.015"
+            radius="0.023" length="0.005" />
     </link>
     <joint name="right_hip" type="revolute">
@@ -626,10 +624,8 @@
         </collision>
         <!-- mass measured with screws -->
-        <inertial>
-            <origin rpy="0 1.5707963267948966 0" xyz="0 0 0.025" />
-            <mass value="0.05267" />
-            <!-- ./cylinder_inertia.py 0.05267 0.025 0.09 -->
-            <inertia ixx="4.37819375e-05" ixy="0" ixz="0" iyx="0" iyy="4.37819375e-05" iyz="0" izx="0" izy="0" izz="1.6459375e-05" />
-        </inertial>
+        <xacro:cylinder_inertia
+            rpy="0 1.5707963267948966 0" xyz="0 0 0.025"
+            mass="0.05267"
+            radius="0.025" length="0.09" />
     </link>
     <joint name="right_hip_horn_fix" type="fixed">
@@ -683,10 +679,8 @@
         </collision>
         <!-- mass based on filament estimate from Prusa Slicer -->
-        <inertial>
-            <origin rpy="0 1.5707963267948966 0" xyz="0.03 0 0" />
-            <mass value="0.09874" />
-            <!-- ./cylinder_inertia.py 0.09874 0.05 0.06 -->
-            <inertia ixx="9.133450000000001e-05" ixy="0" ixz="0" iyx="0" iyy="9.133450000000001e-05" iyz="0" izx="0" izy="0" izz="0.000123425" />
-        </inertial>
+        <xacro:cylinder_inertia
+            rpy="0 1.5707963267948966 0" xyz="0.03 0 0"
+            mass="0.09874"
+            radius="0.05" length="0.06" />
     </link>
     <link name="right_knee_qdd100_stator">
@@ -736,10 +730,8 @@
         </collision>
         <!-- mass guessed from spec -->
-        <inertial>
-            <origin rpy="0 0 0" xyz="0 0 -0.0025" />
-            <mass value="0.015" />
-            <!-- ./cylinder_inertia.py 0.015 0.023 0.005 -->
-            <inertia ixx="2.0149999999999998e-06" ixy="0" ixz="0" iyx="0" iyy="2.0149999999999998e-06" iyz="0" izx="0" izy="0" izz="3.9675e-06" />
-        </inertial>
+        <xacro:cylinder_inertia
+            rpy="0 0 0" xyz="0 0 -0.0025"
+            mass="0.015"
+            radius="0.023" length="0.005" />
     </link>
     <link name="right_knee_horn">
@@ -757,10 +749,8 @@
         </collision>
         <!-- mass measured with screws -->
-        <inertial>
-            <origin rpy="0 1.5707963267948966 0" xyz="0 0 0.025" />
-            <mass value="0.05267" />
-            <!-- ./cylinder_inertia.py 0.05267 0.025 0.09 -->
-            <inertia ixx="4.37819375e-05" ixy="0" ixz="0" iyx="0" iyy="4.37819375e-05" iyz="0" izx="0" izy="0" izz="1.6459375e-05" />
-        </inertial>
+        <xacro:cylinder_inertia
+            rpy="0 1.5707963267948966 0" xyz="0 0 0.025"
+            mass="0.05267"
+            radius="0.025" length="0.09" />
     </link>
     <joint name="right_knee_horn_fix" type="fixed">

Commit message: Move torso to a separate Xacro file
Also, make the handle optional

File: xacro/upkie.xacro (robot description, xacro)
@@ -8,4 +8,5 @@
     <xacro:include filename="xacro/box_inertia.xacro" />
     <xacro:include filename="xacro/cylinder_inertia.xacro" />
+    <xacro:include filename="xacro/torso.xacro" />
     <material name="black">
         <color rgba="0.1 0.1 0.1 1" />
@@ -60,77 +61,5 @@
         <child link="imu" />
     </joint>
-    <!-- Torso -->
-    <link name="torso">
-        <visual>
-            <geometry>
-                <box size="0.125 0.17 0.25" />
-            </geometry>
-            <material name="terracotta_transparent" />
-        </visual>
-        <collision>
-            <geometry>
-                <box size="0.125 0.17 0.25" />
-            </geometry>
-        </collision>
-        <!-- torso mass evaluated as net mass (5.4 [kg]) minus everything else -->
-        <xacro:box_inertia
-            rpy="0 0 0" xyz="0 0 0"
-            mass="1"
-            len_x="0.125" len_y="0.17" len_z="0.25" />
-    </link>
-    <joint name="torso_fix" type="fixed">
-        <origin rpy="0 0 0" xyz="0 0 -0.1" />
-        <parent link="base" />
-        <child link="torso" />
-    </joint>
-    <!-- Battery -->
-    <link name="battery">
-        <visual>
-            <geometry>
-                <box size="0.13 0.074 0.055" />
-            </geometry>
-            <material name="dark_gray" />
-        </visual>
-        <collision>
-            <geometry>
-                <box size="0.13 0.074 0.055" />
-            </geometry>
-        </collision>
-        <!-- mass measurement was imprecise -->
-        <xacro:box_inertia
-            rpy="0 0 0" xyz="0 0 0"
-            mass="0.8"
-            len_x="0.13" len_y="0.074" len_z="0.055" />
-    </link>
-    <joint name="battery_fix" type="fixed">
-        <origin rpy="1.5707963267948966 0 1.5707963267948966" xyz="-0.04 0 0" />
-        <parent link="torso" />
-        <child link="battery" />
-    </joint>
-    <!-- Handle -->
-    <link name="handle">
-        <visual>
-            <geometry>
-                <mesh filename="package://upkie_description/meshes/handle.stl" />
-            </geometry>
-            <material name="terracotta_light" />
-        </visual>
-        <collision>
-            <origin rpy="0 0 0" xyz="0 0 0.01" />
-            <geometry>
-                <box size="0.120 0.07 0.04" />
-            </geometry>
-        </collision>
-        <!-- mass measured on a real robot -->
-        <xacro:box_inertia
-            rpy="0 0 0" xyz="0 0 0.01"
-            mass="0.0525"
-            len_x="0.120" len_y="0.07" len_z="0.04" />
-    </link>
-    <joint name="handle_fix" type="fixed">
-        <origin rpy="0 0 -1.5707963267948966" xyz="0 0 0.135" />
-        <parent link="torso" />
-        <child link="handle" />
-    </joint>
+    <xacro:torso with_camera="false" with_handle="true" />
     <!-- Left leg -->
     <!-- Left hip -->

Commit message: Move materials to a separate file

File: xacro/upkie.xacro (robot description, xacro)
@@ -8,32 +8,6 @@
     <xacro:include filename="xacro/box_inertia.xacro" />
     <xacro:include filename="xacro/cylinder_inertia.xacro" />
+    <xacro:include filename="xacro/materials.xacro" />
     <xacro:include filename="xacro/torso.xacro" />
-    <material name="black">
-        <color rgba="0.1 0.1 0.1 1" />
-    </material>
-    <material name="dark_gray">
-        <color rgba="0.3 0.3 0.3 1" />
-    </material>
-    <material name="light_gray">
-        <color rgba="0.8 0.8 0.8 1" />
-    </material>
-    <material name="light_wood">
-        <color rgba="1 0.77 0.48 1" />
-    </material>
-    <material name="terracotta_light">
-        <color rgba="0.93 0.64 0.52 1" />
-    </material>
-    <material name="terracotta_transparent">
-        <color rgba="0.93 0.64 0.52 0.8" />
-    </material>
-    <material name="chalky_blue">
-        <color rgba="0.65 0.76 0.91 1" />
-    </material>
-    <material name="mj5208_rotor">
-        <color rgba="0.5 0.55 0.6 1.0" />
-    </material>
-    <material name="mj5208_stator">
-        <color rgba="0.22 0.22 0.25 1.0" />
-    </material>
     <link name="base">
         <!-- virtual link -->

Commit message: Move legs to separate Xacro files

File: xacro/upkie.xacro (robot description, xacro)
@@ -12,863 +12,11 @@
     <xacro:include filename="xacro/cylinder_inertia.xacro" />
     <xacro:include filename="xacro/materials.xacro" />
+    <xacro:include filename="xacro/virtual_link_inertia.xacro" />
+    <xacro:include filename="xacro/left_leg.xacro" />
+    <xacro:include filename="xacro/right_leg.xacro" />
     <xacro:include filename="xacro/torso.xacro" />
-    <link name="base">
-        <!-- virtual link -->
-        <inertial>
-            <!-- mass should not be zero [1] -->
-            <mass value="0.001" />
-            <origin rpy="0 0 0" xyz="0 0 0" />
-            <inertia ixx="0" ixy="0" ixz="0" iyy="0" iyz="0" izz="0" />
-        </inertial>
-    </link>
     <xacro:torso with_handle="true" />
-    <!-- Left leg -->
-    <!-- Left hip -->
-    <link name="left_hip_qdd100_stator">
-        <visual>
-            <geometry>
-                <mesh filename="package://upkie_description/meshes/mjbots/qdd100_stator.stl" />
-            </geometry>
-            <material name="black" />
-        </visual>
-        <collision>
-            <origin rpy="0 0 0" xyz="0 0 0.015" />
-            <geometry>
-                <cylinder length="0.03" radius="0.05" />
-            </geometry>
-        </collision>
-        <!-- mass guessed from spec -->
-        <xacro:cylinder_inertia
-            rpy="0 0 0" xyz="0 0 0.015"
-            mass="0.47"
-            radius="0.05" length="0.03" />
-    </link>
-    <joint name="left_hip_qdd100_stator_fix" type="fixed">
-        <origin rpy="-1.5707963267948966 0 0" xyz="0.0 0.085 -0.064" />
-        <parent link="torso" />
-        <child link="left_hip_qdd100_stator" />
-    </joint>
-    <link name="left_hip_qdd100_rotor">
-        <visual>
-            <geometry>
-                <mesh filename="package://upkie_description/meshes/mjbots/qdd100_rotor.stl" />
-            </geometry>
-            <material name="black" />
-        </visual>
-        <collision>
-            <origin rpy="0 0 0" xyz="0 0 -0.0025" />
-            <geometry>
-                <cylinder length="0.005" radius="0.023" />
-            </geometry>
-        </collision>
-        <!-- mass guessed from spec -->
-        <xacro:cylinder_inertia
-            rpy="0 0 0" xyz="0 0 -0.0025"
-            mass="0.015"
-            radius="0.023" length="0.005" />
-    </link>
-    <joint name="left_hip" type="revolute">
-        <parent link="left_hip_qdd100_stator" />
-        <child link="left_hip_qdd100_rotor" />
-        <origin rpy="0 0 0" xyz="0 0 0.0292" />
-        <!-- negative z-axis: search "moteus-direction-configuration" -->
-        <axis xyz="0 0 -1" />
-        <limit effort="16.0" lower="-1.26" upper="1.26" velocity="28.8" />
-    </joint>
-    <link name="left_hip_horn">
-        <visual>
-            <geometry>
-                <mesh filename="package://upkie_description/meshes/mjbots/qdd100_horn.stl" />
-            </geometry>
-            <material name="black" />
-        </visual>
-        <collision>
-            <origin rpy="0 1.5707963267948966 0" xyz="0 0 0.025" />
-            <geometry>
-                <cylinder length="0.09" radius="0.025" />
-            </geometry>
-        </collision>
-        <!-- mass measured with screws -->
-        <xacro:cylinder_inertia
-            rpy="0 1.5707963267948966 0" xyz="0 0 0.025"
-            mass="0.05267"
-            radius="0.025" length="0.09" />
-    </link>
-    <joint name="left_hip_horn_fix" type="fixed">
-        <parent link="left_hip_qdd100_rotor" />
-        <child link="left_hip_horn" />
-        <origin rpy="0 0 1.5707963267948966" xyz="0 0 0" />
-    </joint>
-    <!-- Left femur -->
-    <link name="left_femur">
-        <visual>
-            <geometry>
-                <cylinder length="0.25" radius="0.011" />
-            </geometry>
-            <material name="light_wood" />
-        </visual>
-        <collision>
-            <geometry>
-                <cylinder length="0.26" radius="0.012" />
-            </geometry>
-            <material name="light_wood" />
-        </collision>
-        <!-- mass measured on average over four wooden sticks -->
-        <xacro:cylinder_inertia
-            rpy="0 0 0" xyz="0 0 0"
-            mass="0.056"
-            radius="0.012" length="0.026" />
-    </link>
-    <joint name="left_femur_fix" type="fixed">
-        <parent link="left_hip_qdd100_rotor" />
-        <child link="left_femur" />
-        <origin rpy="1.5707963267948966 0 0" xyz="0 0.07 0.025" />
-    </joint>
-    <!-- Left knee -->
-    <joint name="left_knee_stator_fix" type="fixed">
-        <parent link="left_femur" />
-        <child link="left_knee_stator" />
-        <origin rpy="0 0 -1.5707963267948966" xyz="0 0.042 -0.098" />
-    </joint>
-    <link name="left_knee_stator">
-        <visual>
-            <geometry>
-                <mesh filename="package://upkie_description/meshes/knee_stator.stl" />
-            </geometry>
-            <material name="terracotta_light" />
-        </visual>
-        <collision>
-            <origin rpy="0 1.5707963267948966 0" xyz="0.03 0 0" />
-            <geometry>
-                <cylinder length="0.06" radius="0.05" />
-            </geometry>
-        </collision>
-        <!-- mass based on filament estimate from Prusa Slicer -->
-        <xacro:cylinder_inertia
-            rpy="0 1.5707963267948966 0" xyz="0.03 0 0"
-            mass="0.09874"
-            radius="0.05" length="0.06" />
-    </link>
-    <link name="left_knee_qdd100_stator">
-        <visual>
-            <geometry>
-                <mesh filename="package://upkie_description/meshes/mjbots/qdd100_stator.stl" />
-            </geometry>
-            <material name="black" />
-        </visual>
-        <collision>
-            <origin rpy="0 0 0" xyz="0 0 0.015" />
-            <geometry>
-                <cylinder length="0.03" radius="0.05" />
-            </geometry>
-        </collision>
-        <!-- mass guessed from spec -->
-        <xacro:cylinder_inertia
-            rpy="0 0 0" xyz="0 0 0.015"
-            mass="0.47"
-            radius="0.05" length="0.03" />
-    </link>
-    <joint name="left_knee_qdd100_stator_fix" type="fixed">
-        <parent link="left_knee_stator" />
-        <child link="left_knee_qdd100_stator" />
-        <origin rpy="-1.5707963267948966 0 1.5707963267948966" xyz="0 0 0" />
-    </joint>
-    <joint name="left_knee" type="revolute">
-        <parent link="left_knee_qdd100_stator" />
-        <child link="left_knee_qdd100_rotor" />
-        <origin rpy="0 0 0" xyz="0 0 0.0292" />
-        <!-- negative z-axis: search "moteus-direction-configuration" -->
-        <axis xyz="0 0 -1" />
-        <limit effort="16.0" lower="-2.51" upper="2.51" velocity="28.8" />
-    </joint>
-    <link name="left_knee_qdd100_rotor">
-        <visual>
-            <geometry>
-                <mesh filename="package://upkie_description/meshes/mjbots/qdd100_rotor.stl" />
-            </geometry>
-            <material name="black" />
-        </visual>
-        <collision>
-            <origin rpy="0 0 0" xyz="0 0 -0.0025" />
-            <geometry>
-                <cylinder length="0.005" radius="0.023" />
-            </geometry>
-        </collision>
-        <!-- mass guessed from spec -->
-        <xacro:cylinder_inertia
-            rpy="0 0 0" xyz="0 0 -0.0025"
-            mass="0.015"
-            radius="0.023" length="0.005" />
-    </link>
-    <link name="left_knee_horn">
-        <visual>
-            <geometry>
-                <mesh filename="package://upkie_description/meshes/mjbots/qdd100_horn.stl" />
-            </geometry>
-            <material name="terracotta_light" />
-        </visual>
-        <collision>
-            <origin rpy="0 1.5707963267948966 0" xyz="0 0 0.025" />
-            <geometry>
-                <cylinder length="0.09" radius="0.025" />
-            </geometry>
-        </collision>
-        <!-- mass measured with screws -->
-        <xacro:cylinder_inertia
-            rpy="0 1.5707963267948966 0" xyz="0 0 0.025"
-            mass="0.05267"
-            radius="0.025" length="0.09" />
-    </link>
-    <joint name="left_knee_horn_fix" type="fixed">
-        <parent link="left_knee_qdd100_rotor" />
-        <child link="left_knee_horn" />
-        <origin rpy="0 0 1.5707963267948966" xyz="0 0 0" />
-    </joint>
-    <!-- Left tibia -->
-    <link name="left_tibia">
-        <visual>
-            <geometry>
-                <cylinder length="0.25" radius="0.011" />
-            </geometry>
-            <material name="light_wood" />
-        </visual>
-        <collision>
-            <geometry>
-                <cylinder length="0.26" radius="0.012" />
-            </geometry>
-            <material name="light_wood" />
-        </collision>
-        <!-- mass measured on average over four wooden sticks -->
-        <xacro:cylinder_inertia
-            rpy="0 0 0" xyz="0 0 0"
-            mass="0.056"
-            radius="0.012" length="0.026" />
-    </link>
-    <joint name="left_tibia_fix" type="fixed">
-        <parent link="left_knee_qdd100_rotor" />
-        <child link="left_tibia" />
-        <origin rpy="1.5707963267948966 3.141592653589793 0" xyz="0 0.07 0.025" />
-    </joint>
-    <!-- Left ankle -->
-    <link name="left_ankle_base">
-        <visual>
-            <geometry>
-                <mesh filename="package://upkie_description/meshes/ankle_stator.stl" />
-            </geometry>
-            <material name="chalky_blue" />
-        </visual>
-        <collision>
-            <origin rpy="0 0 0" xyz="0 0.002 0.0275" />
-            <geometry>
-                <box size="0.092 0.068 0.056" />
-            </geometry>
-        </collision>
-        <!-- mass measured with screws -->
-        <xacro:box_inertia
-            rpy="0 0 0" xyz="0 0.002 0.0275"
-            mass="0.07863"
-            len_x="0.092" len_y="0.068" len_z="0.056" />
-    </link>
-    <joint name="left_ankle_base_fix" type="fixed">
-        <parent link="left_tibia" />
-        <child link="left_ankle_base" />
-        <origin rpy="1.5707963267948966 0 0" xyz="0 0.034 -0.105" />
-    </joint>
-    <link name="left_ankle_plate">
-        <visual>
-            <geometry>
-                <box size="0.08 0.045 0.003" />
-            </geometry>
-            <material name="light_gray" />
-        </visual>
-        <collision>
-            <geometry>
-                <box size="0.09 0.046 0.004" />
-            </geometry>
-        </collision>
-        <!-- mass is a pure guess (^_^") -->
-        <xacro:box_inertia
-            rpy="0 0 0" xyz="0 0 0"
-            mass="0.02"
-            len_x="0.09" len_y="0.046" len_z="0.004" />
-    </link>
-    <joint name="left_ankle_plate_fix" type="fixed">
-        <parent link="left_ankle_base" />
-        <child link="left_ankle_plate" />
-        <origin rpy="0 0 0" xyz="0 0 -0.0015" />
-    </joint>
-    <link name="left_ankle_mj5208_stator">
-        <visual>
-            <geometry>
-                <mesh filename="package://upkie_description/meshes/mjbots/mj5208_stator.stl" />
-            </geometry>
-            <material name="mj5208_stator" />
-        </visual>
-        <collision>
-            <origin rpy="0 0 0" xyz="0 0 0.01" />
-            <geometry>
-                <cylinder length="0.018" radius="0.03" />
-            </geometry>
-        </collision>
-        <!-- mass measured was 242.1 [g], minus 20 [g] for the plate, minus 50 [g] for the rotor -->
-        <xacro:cylinder_inertia
-            rpy="0 0 0" xyz="0 0 0.01"
-            mass="0.1721"
-            radius="0.03" length="0.018" />
-    </link>
-    <joint name="left_ankle_mj5208_stator_fix" type="fixed">
-        <parent link="left_ankle_plate" />
-        <child link="left_ankle_mj5208_stator" />
-        <origin rpy="3.141592653589793 0 0" xyz="0 0 -0.0015" />
-    </joint>
-    <link name="left_anchor">
-        <!-- virtual link -->
-        <inertial>
-            <!-- mass should not be zero [1] -->
-            <mass value="0.001" />
-            <origin rpy="0 0 0" xyz="0 0 0" />
-            <inertia ixx="0" ixy="0" ixz="0" iyy="0" iyz="0" izz="0" />
-        </inertial>
-    </link>
-    <joint name="left_anchor_fix" type="fixed">
-        <parent link="left_ankle_mj5208_stator" />
-        <child link="left_anchor" />
-        <origin rpy="1.5707963267948966 3.141592653589793 0" xyz="0 0.0545 0.05" />
-    </joint>
-    <link name="left_ankle_mj5208_rotor">
-        <visual>
-            <geometry>
-                <mesh filename="package://upkie_description/meshes/mjbots/mj5208_rotor.stl" />
-            </geometry>
-            <material name="mj5208_rotor" />
-        </visual>
-        <collision>
-            <origin rpy="0 0 0" xyz="0 0 0.015" />
-            <geometry>
-                <cylinder length="0.016" radius="0.034" />
-            </geometry>
-        </collision>
-        <!-- mass is a pure guess -->
-        <xacro:cylinder_inertia
-            rpy="0 0 0" xyz="0 0 0.015"
-            mass="0.05"
-            radius="0.034" length="0.016" />
-    </link>
-    <joint name="left_wheel" type="revolute">
-        <parent link="left_ankle_mj5208_stator" />
-        <child link="left_ankle_mj5208_rotor" />
-        <origin rpy="0 0 0" xyz="0 0 0" />
-        <!-- negative z-axis: search "moteus-direction-configuration" -->
-        <axis xyz="0 0 -1" />
-        <limit effort="1.7" velocity="111.0" />
-    </joint>
-    <!-- Left wheel -->
-    <link name="left_wheel_hub">
-        <visual>
-            <geometry>
-                <mesh filename="package://upkie_description/meshes/wheel_hub.stl" />
-            </geometry>
-            <material name="terracotta_light" />
-        </visual>
-        <collision>
-            <origin rpy="0 0 0" xyz="0 0 0.0125" />
-            <geometry>
-                <cylinder length="0.025" radius="0.039" />
-            </geometry>
-        </collision>
-        <!-- mass measured with hub adapter -->
-        <xacro:cylinder_inertia
-            rpy="0 0 0" xyz="0 0 0.0125"
-            mass="0.0454"
-            radius="0.039" length="0.025" />
-    </link>
-    <joint name="left_wheel_hub_fix" type="fixed">
-        <parent link="left_ankle_mj5208_rotor" />
-        <child link="left_wheel_hub" />
-        <origin rpy="0 0 0" xyz="0 0 0.0251" />
-    </joint>
-    <link name="left_wheel_tire">
-        <visual>
-            <geometry>
-                <mesh filename="package://upkie_description/meshes/wheel_tire/wheel_tire.stl" />
-            </geometry>
-            <material name="dark_gray" />
-        </visual>
-        <collision>
-            <geometry>
-                <cylinder length="0.04" radius="0.05" />
-            </geometry>
-        </collision>
-        <!-- mass measured on a real robot -->
-        <xacro:cylinder_inertia
-            rpy="0 0 0" xyz="0 0 0"
-            mass="0.08715"
-            radius="0.05" length="0.04" />
-        <contact>
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