Commit message: Use macro for virtual link inertias

File: xacro/right_leg.xacro (robot description, xacro)
@@ -303,11 +303,5 @@
         </joint>
         <link name="right_anchor">
-            <!-- virtual link -->
-            <inertial>
-                <!-- mass should not be zero [1] -->
-                <mass value="0.001" />
-                <origin rpy="0 0 0" xyz="0 0 0" />
-                <inertia ixx="0" ixy="0" ixz="0" iyy="0" iyz="0" izz="0" />
-            </inertial>
+            <xacro:virtual_link_inertia />
         </link>
         <joint name="right_anchor_fix" type="fixed">
@@ -398,11 +392,5 @@
         </joint>
         <link name="right_contact">
-            <!-- virtual link -->
-            <inertial>
-                <!-- mass should not be zero [1] -->
-                <mass value="0.001" />
-                <origin rpy="0 0 0" xyz="0 0 0" />
-                <inertia ixx="0" ixy="0" ixz="0" iyy="0" iyz="0" izz="0" />
-            </inertial>
+            <xacro:virtual_link_inertia />
         </link>
         <joint name="right_contact_fix" type="fixed">
@@ -414,11 +402,5 @@
         </joint>
         <link name="right_wheel_center">
-            <!-- virtual link -->
-            <inertial>
-                <!-- mass should not be zero [1] -->
-                <mass value="0.001" />
-                <origin rpy="0 0 0" xyz="0 0 0" />
-                <inertia ixx="0" ixy="0" ixz="0" iyy="0" iyz="0" izz="0" />
-            </inertial>
+            <xacro:virtual_link_inertia />
         </link>
         <joint name="right_wheel_center_fix" type="fixed">

File: xacro/torso.xacro (robot description, xacro)
@@ -4,11 +4,5 @@
     <xacro:macro name="torso" params="with_handle">
         <link name="base">
-            <!-- virtual link -->
-            <inertial>
-                <!-- mass should not be zero [1] -->
-                <mass value="0.001" />
-                <origin rpy="0 0 0" xyz="0 0 0" />
-                <inertia ixx="0" ixy="0" ixz="0" iyy="0" iyz="0" izz="0" />
-            </inertial>
+            <xacro:virtual_link_inertia />
         </link>
         <!-- Torso -->
