Commit message: Remove with_camera parameter for now

File: xacro/torso.xacro (robot description, xacro)
@@ -2,5 +2,5 @@
 <!-- SPDX-License-Identifier: Apache-2.0 -->
 <robot name="upkie" xmlns:xacro="http://ros.org/wiki/xacro">
-    <xacro:macro name="torso" params="with_camera with_handle">
+    <xacro:macro name="torso" params="with_handle">
         <!-- Torso -->
         <link name="torso">

File: xacro/upkie.xacro (robot description, xacro)
@@ -19,5 +19,5 @@
         </inertial>
     </link>
-    <xacro:torso with_camera="false" with_handle="true" />
+    <xacro:torso with_handle="true" />
     <!-- Left leg -->
     <!-- Left hip -->

Commit message: Move base link to torso.xacro

File: xacro/torso.xacro (robot description, xacro)
@@ -3,4 +3,13 @@
 <robot name="upkie" xmlns:xacro="http://ros.org/wiki/xacro">
     <xacro:macro name="torso" params="with_handle">
+        <link name="base">
+            <!-- virtual link -->
+            <inertial>
+                <!-- mass should not be zero [1] -->
+                <mass value="0.001" />
+                <origin rpy="0 0 0" xyz="0 0 0" />
+                <inertia ixx="0" ixy="0" ixz="0" iyy="0" iyz="0" izz="0" />
+            </inertial>
+        </link>
         <!-- Torso -->
         <link name="torso">
@@ -29,11 +38,5 @@
         <!-- IMU -->
         <link name="imu">
-            <!-- virtual link -->
-            <inertial>
-                <!-- mass should not be zero [1] -->
-                <mass value="0.001" />
-                <origin rpy="0 0 0" xyz="0 0 0" />
-                <inertia ixx="0" ixy="0" ixz="0" iyy="0" iyz="0" izz="0" />
-            </inertial>
+            <xacro:virtual_link_inertia />
         </link>
         <joint name="imu_fix" type="fixed">

Commit message: WIP: Move handle.stl to add-ons directory

File: xacro/torso.xacro (robot description, xacro)
@@ -69,5 +69,5 @@
                 <visual>
                     <geometry>
-                        <mesh filename="package://upkie_description/meshes/handle.stl" />
+                        <mesh filename="package://upkie_description/meshes/add-ons/handle.stl" />
                     </geometry>
                     <material name="terracotta_light" />

Commit message: WIP: Add camera variant

File: xacro/torso.xacro (robot description, xacro)
@@ -2,5 +2,5 @@
 <!-- SPDX-License-Identifier: Apache-2.0 -->
 <robot name="upkie" xmlns:xacro="http://ros.org/wiki/xacro">
-    <xacro:macro name="torso" params="with_handle">
+    <xacro:macro name="torso" params="with_camera with_handle">
         <link name="base">
             <xacro:virtual_link_inertia />
@@ -64,4 +64,31 @@
             <child link="battery" />
         </joint>
+        <xacro:if value="${with_camera}">
+            <!-- Camera -->
+            <link name="camera_support">
+                <visual>
+                    <geometry>
+                        <mesh filename="package://upkie_description/meshes/add-ons/camera_support.stl" />
+                    </geometry>
+                    <material name="terracotta_light" />
+                </visual>
+                <collision>
+                    <origin rpy="0 0 0" xyz="0 0 0" />
+                    <geometry>
+                        <box size="0.11 0.12 0.07" />
+                    </geometry>
+                </collision>
+                <!-- mass NOT MEASURED YET -->
+                <xacro:box_inertia
+                    rpy="0 0 0" xyz="0 0 0"
+                    mass="1.0"
+                    len_x="0.120" len_y="0.07" len_z="0.04" />
+            </link>
+            <joint name="camera_support_fix" type="fixed">
+                <origin rpy="0 0 0" xyz="0 0 0.16" />
+                <parent link="torso" />
+                <child link="camera_support" />
+            </joint>
+        </xacro:if>
         <xacro:if value="${with_handle}">
             <!-- Handle -->

File: xacro/upkie_camera.xacro (robot description, xacro)
@@ -16,5 +16,5 @@
     <xacro:include filename="xacro/right_leg.xacro" />
     <xacro:include filename="xacro/torso.xacro" />
-    <xacro:torso with_camera="false" with_handle="true" />
+    <xacro:torso with_camera="true" with_handle="false" />
     <xacro:left_leg />
     <xacro:right_leg />

Commit message: WIP : added camera to xacro

File: xacro/torso.xacro (robot description, xacro)
@@ -90,4 +90,28 @@
                 <child link="camera_support" />
             </joint>
+            <link name="camera">
+                <visual>
+                    <geometry>
+                        <mesh filename="package://upkie_description/meshes/add-ons/oakd_lite.stl" />
+                    </geometry>
+                    <material name="terracotta_light" />
+                </visual>
+                <collision>
+                    <origin rpy="0 0 0" xyz="0 0 0" />
+                    <geometry>
+                        <box size="0.11 0.12 0.07" />
+                    </geometry>
+                </collision>
+                <!-- mass NOT MEASURED YET -->
+                <xacro:box_inertia
+                    rpy="0 0 0" xyz="0 0 0"
+                    mass="1.0"
+                    len_x="0.120" len_y="0.07" len_z="0.04" />
+            </link>
+            <joint name="camera_fix" type="fixed">
+                <origin rpy="0 0 0" xyz="0 0 0.16" />
+                <parent link="camera_support" />
+                <child link="camera" />
+            </joint>
         </xacro:if>
         <xacro:if value="${with_handle}">

Commit message: Added camera to xacro

File: xacro/torso.xacro (robot description, xacro)
@@ -79,8 +79,8 @@
                     </geometry>
                 </collision>
-                <!-- mass NOT MEASURED YET -->
+                <!-- mass measured with USB cable -->
                 <xacro:box_inertia
                     rpy="0 0 0" xyz="0 0 0"
-                    mass="1.0"
+                    mass="0.167"
                     len_x="0.120" len_y="0.07" len_z="0.04" />
             </link>
@@ -91,27 +91,29 @@
             </joint>
             <link name="camera">
-                <visual>
-                    <geometry>
-                        <mesh filename="package://upkie_description/meshes/add-ons/oakd_lite.stl" />
-                    </geometry>
-                    <material name="terracotta_light" />
-                </visual>
-                <collision>
-                    <origin rpy="0 0 0" xyz="0 0 0" />
-                    <geometry>
-                        <box size="0.11 0.12 0.07" />
-                    </geometry>
-                </collision>
-                <!-- mass NOT MEASURED YET -->
-                <xacro:box_inertia
+	    <visual>
+	      <geometry>
+		<box size="0.0175 0.091 0.028"/>
+	      </geometry>
+	      <material name="light_grey"/>
+	    </visual>
+	    <collision>
+	      <origin rpy="0 0 0" xyz="0 0 0"/>
+	      <geometry>
+		<box size="0.0175 0.091 0.028"/>
+	      </geometry>
+	    </collision>
+	    <inertial>
+	      <origin rpy="0 0 0" xyz="0 0 0"/>
+	      <xacro:box_inertia
                     rpy="0 0 0" xyz="0 0 0"
-                    mass="1.0"
-                    len_x="0.120" len_y="0.07" len_z="0.04" />
-            </link>
-            <joint name="camera_fix" type="fixed">
-                <origin rpy="0 0 0" xyz="0 0 0.16" />
-                <parent link="camera_support" />
-                <child link="camera" />
-            </joint>
+                    mass="0.061"
+                    len_x="0.0175" len_y="0.091" len_z="0.028" />
+	    </inertial>
+	  </link>
+	  <joint name="camera_fix" type="fixed">
+	    <origin rpy="0 0 0" xyz="0.045 0 0"/>
+	    <parent link="camera_support"/>
+	    <child link="camera"/>
+	  </joint>
         </xacro:if>
         <xacro:if value="${with_handle}">

Commit message: Changed camera color to black

File: xacro/torso.xacro (robot description, xacro)
@@ -95,5 +95,5 @@
 		<box size="0.0175 0.091 0.028"/>
 	      </geometry>
-	      <material name="light_gray"/>
+	      <material name="black"/>
 	    </visual>
 	    <collision>

Commit message: Misindentation

File: xacro/torso.xacro (robot description, xacro)
@@ -107,24 +107,24 @@
                     mass="0.061"
                     len_x="0.0175" len_y="0.091" len_z="0.028" />
-    </link>
-    <joint name="camera_fix" type="fixed">
-        <origin rpy="0 0 0" xyz="0.045 0 0"/>
-        <parent link="camera_support"/>
-        <child link="camera"/>
-    </joint>
-    <link name="camera_eye">
-        <xacro:virtual_link_inertia />
-    <visual>
-      <geometry>
-        <box size="0 0 0"/>
-      </geometry>
-      <material name="black"/>
-    </visual>
-  </link>
-  <joint name="camera_eye_fix" type="fixed">
-    <origin rpy="0 0 0" xyz="0.00875 0 0.005"/>
-    <parent link="camera"/>
-    <child link="camera_eye"/>
-  </joint>
+            </link>
+	    <joint name="camera_fix" type="fixed">
+	        <origin rpy="0 0 0" xyz="0.045 0 0"/>
+	        <parent link="camera_support"/>
+	        <child link="camera"/>
+	    </joint>
+	    <link name="camera_eye">
+	        <xacro:virtual_link_inertia />
+	    <visual>
+	      <geometry>
+	        <box size="0 0 0"/>
+	      </geometry>
+	      <material name="black"/>
+	    </visual>
+	  </link>
+	  <joint name="camera_eye_fix" type="fixed">
+	    <origin rpy="0 0 0" xyz="0.00875 0 0.005"/>
+	    <parent link="camera"/>
+	    <child link="camera_eye"/>
+	  </joint>
         </xacro:if>
         <xacro:if value="${with_handle}">

Commit message: Consistent 4-space indentation in camera definition

File: xacro/torso.xacro (robot description, xacro)
@@ -87,40 +87,40 @@
             </joint>
             <link name="camera">
-	    <visual>
-	      <geometry>
-		<box size="0.0175 0.091 0.028"/>
-	      </geometry>
-	      <material name="black"/>
-	    </visual>
-	    <collision>
-	      <origin rpy="0 0 0" xyz="0 0 0"/>
-	      <geometry>
-		<box size="0.0175 0.091 0.028"/>
-	      </geometry>
-	    </collision>
-	      <xacro:box_inertia
+	            <visual>
+                    <geometry>
+                        <box size="0.0175 0.091 0.028"/>
+                    </geometry>
+                    <material name="black"/>
+                </visual>
+                <collision>
+                    <origin rpy="0 0 0" xyz="0 0 0"/>
+                    <geometry>
+                        <box size="0.0175 0.091 0.028"/>
+                    </geometry>
+                </collision>
+                <xacro:box_inertia
                     rpy="0 0 0" xyz="0 0 0"
                     mass="0.061"
                     len_x="0.0175" len_y="0.091" len_z="0.028" />
             </link>
-	    <joint name="camera_fix" type="fixed">
-	        <origin rpy="0 0 0" xyz="0.045 0 0"/>
-	        <parent link="camera_support"/>
-	        <child link="camera"/>
-	    </joint>
-	    <link name="camera_eye">
-	        <xacro:virtual_link_inertia />
-	    <visual>
-	      <geometry>
-	        <box size="0 0 0"/>
-	      </geometry>
-	      <material name="black"/>
-	    </visual>
-	  </link>
-	  <joint name="camera_eye_fix" type="fixed">
-	    <origin rpy="0 0 0" xyz="0.00875 0 0.005"/>
-	    <parent link="camera"/>
-	    <child link="camera_eye"/>
-	  </joint>
+            <joint name="camera_fix" type="fixed">
+                <origin rpy="0 0 0" xyz="0.045 0 0"/>
+                <parent link="camera_support"/>
+                <child link="camera"/>
+            </joint>
+            <link name="camera_eye">
+                <xacro:virtual_link_inertia />
+                <visual>
+                    <geometry>
+                        <box size="0 0 0"/>
+                    </geometry>
+                    <material name="black"/>
+                </visual>
+            </link>
+            <joint name="camera_eye_fix" type="fixed">
+                <origin rpy="0 0 0" xyz="0.00875 0 0.005"/>
+                <parent link="camera"/>
+                <child link="camera_eye"/>
+            </joint>
         </xacro:if>
         <xacro:if value="${with_handle}">

Commit message: Update camera_eye to virtual_link macro

File: xacro/torso.xacro (robot description, xacro)
@@ -109,13 +109,5 @@
                 <child link="camera"/>
             </joint>
-            <link name="camera_eye">
-                <xacro:virtual_link_inertia />
-                <visual>
-                    <geometry>
-                        <box size="0 0 0"/>
-                    </geometry>
-                    <material name="black"/>
-                </visual>
-            </link>
+            <xacro:virtual_link name="camera_eye" />
             <joint name="camera_eye_fix" type="fixed">
                 <origin rpy="0 0 0" xyz="0.00875 0 0.005"/>
