Commit message: Updated upkie_camera

File: urdf/upkie_camera.urdf (robot description, URDF)
Before this commit: robot upkie, 41 links, 40 joints
Links:
- added link camera, mass 1.0; collision box size=0.11 0.12 0.07; visual mesh filename=package://upkie_description/meshes/add-ons/oakd_lite.stl
Joints:
- added joint camera_fix: type fixed, parent camera_support, child camera, origin xyz=0 0 0.16 rpy=0 0 0

Commit message: updated urdf

File: urdf/upkie_camera.urdf (robot description, URDF)
Before this commit: robot upkie, 42 links, 41 joints
Links:
- link camera: mass 1.0 -> None; geometry collision box size=0.0175 0.091 0.028; visual box size=0.0175 0.091 0.028
- link camera_support: mass 1.0 -> 0.167
Joints:
- joint camera_fix: origin xyz=0 0 0.16 rpy=0 0 0 -> xyz=0.045 0 0 rpy=0 0 0

Commit message: Wrong syntax in torso xacro

File: urdf/upkie_camera.urdf (robot description, URDF)
Before this commit: robot upkie, 42 links, 41 joints
Links:
- link camera: mass None -> 0.061

File: xacro/torso.xacro (robot description, xacro)
@@ -95,5 +95,5 @@
 		<box size="0.0175 0.091 0.028"/>
 	      </geometry>
-	      <material name="light_grey"/>
+	      <material name="light_gray"/>
 	    </visual>
 	    <collision>
@@ -103,11 +103,8 @@
 	      </geometry>
 	    </collision>
-	    <inertial>
-	      <origin rpy="0 0 0" xyz="0 0 0"/>
 	      <xacro:box_inertia
                     rpy="0 0 0" xyz="0 0 0"
                     mass="0.061"
                     len_x="0.0175" len_y="0.091" len_z="0.028" />
-	    </inertial>
 	  </link>
 	  <joint name="camera_fix" type="fixed">

Commit message: Added virtual camera eye frame

File: urdf/upkie_camera.urdf (robot description, URDF)
Before this commit: robot upkie, 42 links, 41 joints
Links:
- added link camera_eye, mass 0.001
Joints:
- added joint camera_eye_fix: type fixed, parent camera, child camera_eye, origin xyz=0.00875 0 0.005 rpy=0 0 0

File: xacro/torso.xacro (robot description, xacro)
@@ -107,10 +107,18 @@
                     mass="0.061"
                     len_x="0.0175" len_y="0.091" len_z="0.028" />
-	  </link>
-	  <joint name="camera_fix" type="fixed">
-	    <origin rpy="0 0 0" xyz="0.045 0 0"/>
-	    <parent link="camera_support"/>
-	    <child link="camera"/>
-	  </joint>
+    </link>
+    <joint name="camera_fix" type="fixed">
+        <origin rpy="0 0 0" xyz="0.045 0 0"/>
+        <parent link="camera_support"/>
+        <child link="camera"/>
+    </joint>
+    <link name="camera_eye">
+        <xacro:virtual_link_inertia />
+    </link>
+    <joint name="camera_eye_fix" type="fixed">
+        <origin rpy="0 0 0" xyz="0.00875 0 0.005"/>
+        <parent link="camera"/>
+        <child link="camera_eye"/>
+    </joint>
         </xacro:if>
         <xacro:if value="${with_handle}">

Commit message: Corrected camera eye position

File: urdf/upkie_camera.urdf (robot description, URDF)
Before this commit: robot upkie, 43 links, 42 joints
Joints:
- joint camera_eye_fix: origin xyz=0.00875 0 0.005 rpy=0 0 0 -> xyz=-0.045 0 0.005 rpy=0 0 0

File: xacro/torso.xacro (robot description, xacro)
@@ -117,5 +117,5 @@
     </link>
     <joint name="camera_eye_fix" type="fixed">
-        <origin rpy="0 0 0" xyz="0.00875 0 0.005"/>
+        <origin rpy="0 0 0" xyz="-0.045 0 0.005"/>
         <parent link="camera"/>
         <child link="camera_eye"/>

Commit message: Corrected camera position and added a zero dimension visual box

File: urdf/upkie_camera.urdf (robot description, URDF)
Before this commit: robot upkie, 43 links, 42 joints
Links:
- link camera_eye: geometry visual box size=0 0 0
Joints:
- joint camera_eye_fix: origin xyz=-0.045 0 0.005 rpy=0 0 0 -> xyz=0.00875 0 0.005 rpy=0 0 0

File: xacro/torso.xacro (robot description, xacro)
@@ -115,10 +115,16 @@
     <link name="camera_eye">
         <xacro:virtual_link_inertia />
-    </link>
-    <joint name="camera_eye_fix" type="fixed">
-        <origin rpy="0 0 0" xyz="-0.045 0 0.005"/>
-        <parent link="camera"/>
-        <child link="camera_eye"/>
-    </joint>
+    <visual>
+      <geometry>
+        <box size="0 0 0"/>
+      </geometry>
+      <material name="black"/>
+    </visual>
+  </link>
+  <joint name="camera_eye_fix" type="fixed">
+    <origin rpy="0 0 0" xyz="0.00875 0 0.005"/>
+    <parent link="camera"/>
+    <child link="camera_eye"/>
+  </joint>
         </xacro:if>
         <xacro:if value="${with_handle}">
