Commit message: Fix IMU orientation according to the pi3hat convention
See https://github.com/tasts-robots/upkie_description/issues/2

pi3hat convention:
    https://github.com/mjbots/pi3hat/blob/master/docs/reference.md#orientation

File: urdf/upkie.urdf (robot description, URDF)
Before this commit: robot upkie, 39 links, 38 joints
Joints:
- joint imu_fix: origin xyz=0 0 0 rpy=0 0 3.141592653589793 -> xyz=0 0 0 rpy=3.141592653589793 0 3.141592653589793

Commit message: Fix the IMU orientation (bis repetita placent)
When Upkie is standing:

- Raspberry Pi -> pi3hat is looking down, so +z is aiming down
- USB ports on the Raspberry Pi are to the right of the robot

Thus in fine the x-axis is pointing forward.

File: urdf/upkie.urdf (robot description, URDF)
Before this commit: robot upkie, 39 links, 38 joints
Joints:
- joint imu_fix: origin xyz=0 0 0 rpy=3.141592653589793 0 3.141592653589793 -> xyz=0 0 0 rpy=3.141592653589793 0 0

Commit message: Update velocity limits to more reasonable values

File: urdf/upkie.urdf (robot description, URDF)
Before this commit: robot upkie, 39 links, 38 joints
Joints:
- joint left_hip: limit lower=-1.54 upper=1.54 effort=10.0 velocity=0.7 -> lower=-1.54 upper=1.54 effort=10.0 velocity=12.0
- joint left_knee: limit lower=-2.57 upper=2.57 effort=10.0 velocity=0.7 -> lower=-2.57 upper=2.57 effort=10.0 velocity=12.0
- joint left_wheel: limit effort=1.0 velocity=0.7 -> effort=1.0 velocity=100.0
- joint right_hip: limit lower=-1.54 upper=1.54 effort=10.0 velocity=0.7 -> lower=-1.54 upper=1.54 effort=10.0 velocity=12.0
- joint right_knee: limit lower=-2.57 upper=2.57 effort=10.0 velocity=0.7 -> lower=-2.57 upper=2.57 effort=10.0 velocity=12.0
- joint right_wheel: limit effort=1.0 velocity=0.7 -> effort=1.0 velocity=100.0

Commit message: Update hip and knee position limits

File: urdf/upkie.urdf (robot description, URDF)
Before this commit: robot upkie, 39 links, 38 joints
Joints:
- joint left_hip: limit lower=-1.54 upper=1.54 effort=10.0 velocity=12.0 -> lower=-1.2566370614359172 upper=1.2566370614359172 effort=10.0 velocity=12.566370614359172
- joint left_knee: limit lower=-2.57 upper=2.57 effort=10.0 velocity=12.0 -> lower=-2.5132741228718345 upper=2.5132741228718345 effort=10.0 velocity=12.0
- joint right_hip: limit lower=-1.54 upper=1.54 effort=10.0 velocity=12.0 -> lower=-1.2566370614359172 upper=1.2566370614359172 effort=10.0 velocity=12.566370614359172
- joint right_knee: limit lower=-2.57 upper=2.57 effort=10.0 velocity=12.0 -> lower=-2.5132741228718345 upper=2.5132741228718345 effort=10.0 velocity=12.0

Commit message: Update wheel velocity limits

File: urdf/upkie.urdf (robot description, URDF)
Before this commit: robot upkie, 39 links, 38 joints
Joints:
- joint left_wheel: limit effort=1.0 velocity=100.0 -> effort=1.0 velocity=50.26548245743669
- joint right_wheel: limit effort=1.0 velocity=100.0 -> effort=1.0 velocity=50.26548245743669

Commit message: Update knee velocity limits

File: urdf/upkie.urdf (robot description, URDF)
Before this commit: robot upkie, 39 links, 38 joints
Joints:
- joint left_knee: limit lower=-2.5132741228718345 upper=2.5132741228718345 effort=10.0 velocity=12.0 -> lower=-2.5132741228718345 upper=2.5132741228718345 effort=10.0 velocity=12.566370614359172
- joint right_knee: limit lower=-2.5132741228718345 upper=2.5132741228718345 effort=10.0 velocity=12.0 -> lower=-2.5132741228718345 upper=2.5132741228718345 effort=10.0 velocity=12.566370614359172

Commit message: Update IMU orientation

File: urdf/upkie.urdf (robot description, URDF)
Before this commit: robot upkie, 39 links, 38 joints
Joints:
- joint imu_fix: origin xyz=0 0 0 rpy=3.141592653589793 0 0 -> xyz=0 0 0 rpy=3.141592653589793 0 3.141592653589793

Commit message: Increase velocity and torque limits to motor specs

File: urdf/upkie.urdf (robot description, URDF)
Before this commit: robot upkie, 41 links, 40 joints
Joints:
- joint left_hip: limit lower=-1.2566370614359172 upper=1.2566370614359172 effort=10.0 velocity=12.566370614359172 -> lower=-1.26 upper=1.26 effort=16.0 velocity=28.8
- joint left_knee: limit lower=-2.5132741228718345 upper=2.5132741228718345 effort=10.0 velocity=12.566370614359172 -> lower=-2.51 upper=2.51 effort=16.0 velocity=28.8
- joint left_wheel: limit effort=1.0 velocity=50.26548245743669 -> effort=1.7 velocity=785.4
- joint right_hip: limit lower=-1.2566370614359172 upper=1.2566370614359172 effort=10.0 velocity=12.566370614359172 -> lower=-1.26 upper=1.26 effort=16.0 velocity=28.8
- joint right_knee: limit lower=-2.5132741228718345 upper=2.5132741228718345 effort=10.0 velocity=12.566370614359172 -> lower=-2.51 upper=2.51 effort=16.0 velocity=28.8
- joint right_wheel: limit effort=1.0 velocity=50.26548245743669 -> effort=1.7 velocity=785.4

Commit message: Allow frame name filtering in example

File: urdf/upkie.urdf (robot description, URDF)
Before this commit: robot upkie, 39 links, 38 joints
Links:
- added link left_anchor, mass 0.01; collision box size=0.01 0.01 0.01; visual box size=0.01 0.01 0.01
- added link right_anchor, mass 0.01; collision box size=0.01 0.01 0.01; visual box size=0.01 0.01 0.01
Joints:
- added joint left_anchor_fix: type fixed, parent left_ankle_mj5208_stator, child left_anchor, origin xyz=0 0.0545 0.05 rpy=1.5707963267948966 3.141592653589793 0
- added joint right_anchor_fix: type fixed, parent right_ankle_mj5208_stator, child right_anchor, origin xyz=0 0.0545 0.048 rpy=1.5707963267948966 0 0

Commit message: Lower and explain maximum wheel velocity

File: urdf/upkie.urdf (robot description, URDF)
Before this commit: robot upkie, 41 links, 40 joints
Joints:
- joint left_wheel: limit effort=1.7 velocity=785.4 -> effort=1.7 velocity=111.0
- joint right_wheel: limit effort=1.7 velocity=785.4 -> effort=1.7 velocity=111.0

Commit message: Remove collision volumes from virtual links

File: urdf/upkie.urdf (robot description, URDF)
Before this commit: robot upkie, 41 links, 40 joints
Links:
- link imu: mass 0.001 -> 0; geometry 
- link left_anchor: mass 0.01 -> 0; geometry 
- link left_contact: mass 0.01 -> 0; geometry 
- link left_wheel_center: mass 0.01 -> 0; geometry 
- link right_anchor: mass 0.01 -> 0; geometry 
- link right_contact: mass 0.01 -> 0; geometry 
- link right_wheel_center: mass 0.01 -> 0; geometry 

Commit message: Make base a virtual link

File: urdf/upkie.urdf (robot description, URDF)
Before this commit: robot upkie, 41 links, 40 joints
Links:
- link base: mass 0.001 -> 0; geometry 

Commit message: Revert "Make base a virtual link"
This reverts commit f3d10f7da4c56c3a828f1c065f100ceb2b726c21.

It removes the robot's floating-base in Bullet.

File: urdf/upkie.urdf (robot description, URDF)
Before this commit: robot upkie, 41 links, 40 joints
Links:
- link base: mass 0 -> 0.001; geometry collision box size=0.01 0.01 0.01; visual box size=0.01 0.001 0.001

Commit message: WIP: Zero out the base inertia only

File: urdf/upkie.urdf (robot description, URDF)
Before this commit: robot upkie, 41 links, 40 joints
Links:
- link base: mass 0.001 -> 0

Commit message: Use non-zero masses for virtual links (Bullet)

File: urdf/upkie.urdf (robot description, URDF)
Before this commit: robot upkie, 41 links, 40 joints
Links:
- link base: mass 0 -> 0.001
- link imu: mass 0 -> 0.001
- link left_anchor: mass 0 -> 0.001
- link left_contact: mass 0 -> 0.001
- link left_wheel_center: mass 0 -> 0.001
- link right_anchor: mass 0 -> 0.001
- link right_contact: mass 0 -> 0.001
- link right_wheel_center: mass 0 -> 0.001

Commit message: Remove collision and visual of base link

File: urdf/upkie.urdf (robot description, URDF)
Before this commit: robot upkie, 41 links, 40 joints
Links:
- link base: geometry 

Commit message: WIP: Generate box inertias from xacro

File: urdf/upkie.urdf (robot description, URDF)
Before this commit: robot upkie, 41 links, 40 joints
Links:
- link torso: mass 1.0 -> 1

File: xacro/upkie.xacro (robot description, xacro)
@@ -5,5 +5,6 @@
 <!-- This file was generated from upkie.xacro -->
 <!-- Conventions in this file are detailed in: https://github.com/upkie/upkie_description/wiki/ -->
-<robot name="upkie">
+<robot name="upkie" xmlns:xacro="http://ros.org/wiki/xacro">
+    <xacro:include filename="xacro/box_inertia.xacro" />
     <material name="black">
         <color rgba="0.1 0.1 0.1 1" />
@@ -71,10 +72,6 @@
             </geometry>
         </collision>
-        <inertial>
-            <!-- torso mass evaluated as net mass (5.4 [kg]) minus everything else -->
-            <mass value="1.0" />
-            <!-- ./box_inertia.py 1.0 0.125 0.17 0.25 -->
-            <inertia ixx="0.007616666666666667" ixy="0" ixz="0" iyx="0" iyy="0.006510416666666666" iyz="0" izx="0" izy="0" izz="0.0037104166666666674" />
-        </inertial>
+        <!-- torso mass evaluated as net mass (5.4 [kg]) minus everything else -->
+        <xacro:box_inertia mass="1" len_x="0.125" len_y="0.17" len_z="0.25" />
     </link>
     <joint name="torso_fix" type="fixed">

Commit message: Change parent of "imu" frame from "base" to "torso"

File: urdf/upkie.urdf (robot description, URDF)
Before this commit: robot upkie, 41 links, 40 joints
Joints:
- joint imu_fix: parent base -> torso

File: xacro/torso.xacro (robot description, xacro)
@@ -26,4 +26,20 @@
             <parent link="base" />
             <child link="torso" />
+        </joint>
+        <!-- IMU -->
+        <link name="imu">
+            <!-- virtual link -->
+            <inertial>
+                <!-- mass should not be zero [1] -->
+                <mass value="0.001" />
+                <origin rpy="0 0 0" xyz="0 0 0" />
+                <inertia ixx="0" ixy="0" ixz="0" iyy="0" iyz="0" izz="0" />
+            </inertial>
+        </link>
+        <joint name="imu_fix" type="fixed">
+            <!-- not that the origin frame is not translated -->
+            <origin rpy="3.141592653589793 0 3.141592653589793" xyz="0 0 0" />
+            <parent link="torso" />
+            <child link="imu" />
         </joint>
         <!-- Battery -->

File: xacro/upkie.xacro (robot description, xacro)
@@ -45,20 +45,4 @@
         </inertial>
     </link>
-    <!-- IMU -->
-    <link name="imu">
-        <!-- virtual link -->
-        <inertial>
-            <!-- mass should not be zero [1] -->
-            <mass value="0.001" />
-            <origin rpy="0 0 0" xyz="0 0 0" />
-            <inertia ixx="0" ixy="0" ixz="0" iyy="0" iyz="0" izz="0" />
-        </inertial>
-    </link>
-    <joint name="imu_fix" type="fixed">
-        <!-- not that the origin frame is not translated -->
-        <origin rpy="3.141592653589793 0 3.141592653589793" xyz="0 0 0" />
-        <parent link="base" />
-        <child link="imu" />
-    </joint>
     <xacro:torso with_camera="false" with_handle="true" />
     <!-- Left leg -->

Commit message: python: Add "variant" keyword argument to `load_in_pinocchio`

File: urdf/upkie.urdf (robot description, URDF)
Before this commit: robot upkie, 41 links, 40 joints
Links:
- link handle: geometry collision box size=0.120 0.07 0.04; visual mesh filename=package://upkie_description/meshes/add-ons/handle.stl

File: urdf/upkie_camera.urdf (robot description, URDF)
Before this commit: robot upkie, 41 links, 40 joints
Links:
- link camera_support: geometry collision box size=0.11 0.12 0.07; visual mesh filename=package://upkie_description/meshes/add-ons/camera_support.s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

Commit message: Add an empty visual box to all virtual links
See https://github.com/upkie/upkie_description/pull/19#issuecomment-2259933854

Fixes https://github.com/upkie/upkie_description/issues/20

File: urdf/upkie.urdf (robot description, URDF)
Before this commit: robot upkie, 41 links, 40 joints
Links:
- link base: geometry visual box size=0 0 0
- link imu: geometry visual box size=0 0 0
- link left_anchor: geometry visual box size=0 0 0
- link left_contact: geometry visual box size=0 0 0
- link left_wheel_center: geometry visual box size=0 0 0
- link right_anchor: geometry visual box size=0 0 0
- link right_contact: geometry visual box size=0 0 0
- link right_wheel_center: geometry visual box size=0 0 0

File: urdf/upkie_camera.urdf (robot description, URDF)
Before this commit: robot upkie, 43 links, 42 joints
Links:
- link base: geometry visual box size=0 0 0
- link imu: geometry visual box size=0 0 0
- link left_anchor: geometry visual box size=0 0 0
- link left_contact: geometry visual box size=0 0 0
- link left_wheel_center: geometry visual box size=0 0 0
- link right_anchor: geometry visual box size=0 0 0
- link right_contact: geometry visual box size=0 0 0
- link right_wheel_center: geometry visual box size=0 0 0

File: xacro/left_leg.xacro (robot description, xacro)
@@ -302,7 +302,5 @@
             <origin rpy="3.141592653589793 0 0" xyz="0 0 -0.0015" />
         </joint>
-        <link name="left_anchor">
-            <xacro:virtual_link_inertia />
-        </link>
+        <xacro:virtual_link name="left_anchor" />
         <joint name="left_anchor_fix" type="fixed">
             <parent link="left_ankle_mj5208_stator" />
@@ -391,7 +389,5 @@
             <origin rpy="0 0 0" xyz="0 0 0.0209" />
         </joint>
-        <link name="left_contact">
-            <xacro:virtual_link_inertia />
-        </link>
+        <xacro:virtual_link name="left_contact" />
         <joint name="left_contact_fix" type="fixed">
             <parent link="left_wheel_tire" />
@@ -401,7 +397,5 @@
             <origin rpy="1.5707963267948966 0 0" xyz="0 0.047 0" />
         </joint>
-        <link name="left_wheel_center">
-            <xacro:virtual_link_inertia />
-        </link>
+        <xacro:virtual_link name="left_wheel_center" />
         <joint name="left_wheel_center_fix" type="fixed">
             <parent link="left_wheel_tire" />

File: xacro/right_leg.xacro (robot description, xacro)
@@ -302,7 +302,5 @@
             <origin rpy="3.141592653589793 0 0" xyz="0 0 -0.0015" />
         </joint>
-        <link name="right_anchor">
-            <xacro:virtual_link_inertia />
-        </link>
+        <xacro:virtual_link name="right_anchor" />
         <joint name="right_anchor_fix" type="fixed">
             <parent link="right_ankle_mj5208_stator" />
@@ -391,7 +389,5 @@
             <origin rpy="0 0 0" xyz="0 0 0.0209" />
         </joint>
-        <link name="right_contact">
-            <xacro:virtual_link_inertia />
-        </link>
+        <xacro:virtual_link name="right_contact" />
         <joint name="right_contact_fix" type="fixed">
             <parent link="right_wheel_tire" />
@@ -401,7 +397,5 @@
             <origin rpy="1.5707963267948966 0 0" xyz="0 0.047 0" />
         </joint>
-        <link name="right_wheel_center">
-            <xacro:virtual_link_inertia />
-        </link>
+        <xacro:virtual_link name="right_wheel_center" />
         <joint name="right_wheel_center_fix" type="fixed">
             <parent link="right_wheel_tire" />

File: xacro/torso.xacro (robot description, xacro)
@@ -3,7 +3,5 @@
 <robot name="upkie" xmlns:xacro="http://ros.org/wiki/xacro">
     <xacro:macro name="torso" params="with_camera with_handle">
-        <link name="base">
-            <xacro:virtual_link_inertia />
-        </link>
+        <xacro:virtual_link name="base" />
         <!-- Torso -->
         <link name="torso">
@@ -31,7 +29,5 @@
         </joint>
         <!-- IMU -->
-        <link name="imu">
-            <xacro:virtual_link_inertia />
-        </link>
+        <xacro:virtual_link name="imu" />
         <joint name="imu_fix" type="fixed">
             <!-- not that the origin frame is not translated -->

File: xacro/upkie.xacro (robot description, xacro)
@@ -12,5 +12,5 @@
     <xacro:include filename="xacro/utils/cylinder_inertia.xacro" />
     <xacro:include filename="xacro/utils/materials.xacro" />
-    <xacro:include filename="xacro/utils/virtual_link_inertia.xacro" />
+    <xacro:include filename="xacro/utils/virtual_link.xacro" />
     <xacro:include filename="xacro/left_leg.xacro" />
     <xacro:include filename="xacro/right_leg.xacro" />

File: xacro/upkie_camera.xacro (robot description, xacro)
@@ -12,5 +12,5 @@
     <xacro:include filename="xacro/utils/cylinder_inertia.xacro" />
     <xacro:include filename="xacro/utils/materials.xacro" />
-    <xacro:include filename="xacro/utils/virtual_link_inertia.xacro" />
+    <xacro:include filename="xacro/utils/virtual_link.xacro" />
     <xacro:include filename="xacro/left_leg.xacro" />
     <xacro:include filename="xacro/right_leg.xacro" />
